File: esc/supplies.kicad_sch (KiCad schematic)
At the start: 26 parts

Commit message: Finished layout
Parts:
- removed L?: L, symbol Device:L
- added C17: 470u, Capacitor_THT:CP_Radial_D10.0mm_P5.00mm, symbol Device:C_Polarized
- added C47: 1u, Capacitor_SMD:C_0603_1608Metric, symbol Device:C
- added L3: 100u, Inductor_SMD:L_Sumida_CR75, symbol Device:L
- added NT2: NetTie_2, footprints:Nettie2, symbol Device:NetTie_2
- added SW2, SW3: SW_SPDT, Connector_PinHeader_2.54mm:PinHeader_1x03_P2.54mm_Vertical, symbol Switch:SW_SPDT
- C14: renamed from C?; footprint (none) -> Capacitor_THT:CP_Radial_D10.0mm_P5.00mm
- C15: renamed from C?; footprint (none) -> Capacitor_SMD:C_0603_1608Metric
- C16: renamed from C?; value 100u -> 220u; footprint (none) -> Capacitor_THT:CP_Radial_D8.0mm_P3.50mm
- C18: renamed from C?; value C -> 470p; footprint (none) -> Capacitor_SMD:C_0603_1608Metric
- C19, C20, C21: renamed from C?; value C -> 10u; footprint (none) -> Capacitor_SMD:C_0805_2012Metric
- C22: renamed from C?; value C_Polarized -> 220u; footprint (none) -> Capacitor_THT:CP_Radial_D8.0mm_P3.50mm
- D1, D2: renamed from D?; value D -> SS14; footprint (none) -> Diode_SMD:D_SMA
- L1: renamed from L?; footprint (none) -> Inductor_SMD:L_Sumida_CR75
- L2: renamed from L?; value L -> 100u; footprint (none) -> Inductor_SMD:L_Sumida_CR75
- NT1: renamed from NT?; footprint (none) -> footprints:Nettie3
- R24: renamed from R?; value 0.5 -> 0.51; footprint (none) -> Resistor_SMD:R_1206_3216Metric
- R25, R26, R30: renamed from R?; footprint (none) -> Resistor_SMD:R_0603_1608Metric
- R27: renamed from R?; value 0.33 -> 0.51; footprint (none) -> Resistor_SMD:R_1206_3216Metric
- R28: renamed from R?; value R -> 1k; footprint (none) -> Resistor_SMD:R_0603_1608Metric
- R29: renamed from R?; value R -> 180; footprint (none) -> Resistor_SMD:R_0603_1608Metric
- R31: renamed from R?; value R -> 13k; footprint (none) -> Resistor_SMD:R_0603_1608Metric
- R32: renamed from R?; value R -> 1.5k; footprint (none) -> Resistor_SMD:R_0603_1608Metric
- gave numbers to parts that had none: 3
Connections:
- net +12V: now also SW3.2 (B); no longer C22.1, D2.1 (K), R31.1
- net +3.3VA: now also C47.1, NT2.2
- net +3V3: now also NT2.1
- net GND: now also C17.2
- net GNDA: now also C47.2
- net at D1.1 (K), U4.2 (SwE): now also L3.1; no longer L1.1
- net +5V: now reaches C19.1, R27.1, U5.6 (Vin), U6.3 (VI)
- net +5V: now also C17.1, SW2.2 (B); no longer C16.1, L1.2, R25.1
- net VIN: now reaches C14.1, R24.1, U4.6 (Vin)
- net VIN: now also SW2.3 (C), SW3.3 (C)
- new net: L1.1, L3.2
- new net: C16.1, L1.2, R25.1, SW2.1 (A)
- new net: C22.1, D2.1 (K), R31.1, SW3.1 (A)
Other:
- note added: "12V supply"
- note added: "3V3 supply"
- note added: "5V supply"
- note added: "Ground star point"
- note added: "t_{on,max} = C_{T} / 4e-5 = 1.18e-5s t_{off,min} = 2e-6s T = 1.38e-5s f = 72.5kHz V_{in} = 5V V_{sat} = ~1V V_{out} = 12V I_{out,max} = 0.1A -(V_{in} - V_{sat}) t_{on} = (V_{in} - V_{out} - V_{f}) t_{off} t_{on} / t_{off} = (V_{out} - V_{in} + V_{f}) / (V_{in} - V_{sat}) = r = 1.93 t_{on} = r t_{off} T = t_{on} + t_{off} = (r + 1) t_{off} Assuming continuous operation at I_{out,max}, the maximum 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"
- note removed: "5V"
- moved on the sheet: C14, C15, C16, C18, C19, C20, C21, C22, D1, D2, L1, L2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

Commit message: Finished design - first submission
Parts:
- added TP16, TP17, TP18, TP19, TP20, TP21: TestPoint, symbol Connector:TestPoint
Connections:
- net +12V: now also TP21.1
- net +3.3VA: now also TP20.1
- net +3V3: now also TP19.1
- net +5V: now also TP17.1
- net GND: now also TP16.1
- net GNDA: now also TP18.1
Changed lines of the file:
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@@
   (junction (at 103.505 66.04) (diameter 0) (color 0 0 0 0)
   )
+  (junction (at 250.19 120.015) (diameter 0) (color 0 0 0 0)
+  )
   (junction (at 66.675 60.325) (diameter 0) (color 0 0 0 0)
   )
   (junction (at 173.355 48.26) (diameter 0) (color 0 0 0 0)
   )
+  (junction (at 131.445 156.21) (diameter 0) (color 0 0 0 0)
+  )
   (junction (at 114.935 55.88) (diameter 0) (color 0 0 0 0)
   )
@@
   (junction (at 103.505 55.88) (diameter 0) (color 0 0 0 0)
   )
+  (junction (at 137.795 152.4) (diameter 0) (color 0 0 0 0)
+  )
   (junction (at 222.25 56.515) (diameter 0) (color 0 0 0 0)
   )
@@
   (junction (at 31.115 57.785) (diameter 0) (color 0 0 0 0)
   )
+  (junction (at 134.62 53.34) (diameter 0) (color 0 0 0 0)
+  )
   (junction (at 245.745 120.015) (diameter 0) (color 0 0 0 0)
   )
+  (junction (at 276.86 50.165) (diameter 0) (color 0 0 0 0)
+  )
+  (junction (at 226.695 120.015) (diameter 0) (color 0 0 0 0)
+  )
   (junction (at 250.825 59.055) (diameter 0) (color 0 0 0 0)
   )
@@
     (stroke (width 0) (type default) (color 0 0 0 0))
   )
-  (wire (pts (xy 247.65 120.015) (xy 254 120.015))
+  (wire (pts (xy 247.65 120.015) (xy 250.19 120.015))
     (stroke (width 0) (type default) (color 0 0 0 0))
   )
@@
     (stroke (width 0) (type default) (color 0 0 0 0))
   )
-  (wire (pts (xy 131.445 155.575) (xy 131.445 156.845))
+  (wire (pts (xy 131.445 155.575) (xy 131.445 156.21))
     (stroke (width 0) (type default) (color 0 0 0 0))
   )
@@
     (stroke (width 0) (type default) (color 0 0 0 0))
   )
+  (wire (pts (xy 226.695 120.015) (xy 229.235 120.015))
+    (stroke (width 0) (type default) (color 0 0 0 0))
+  )
   (wire (pts (xy 101.6 55.88) (xy 103.505 55.88))
     (stroke (width 0) (type default) (color 0 0 0 0))
@@
     (stroke (width 0) (type default) (color 0 0 0 0))
   )
+  (wire (pts (xy 131.445 156.21) (xy 131.445 156.845))
+    (stroke (width 0) (type default) (color 0 0 0 0))
+  )
   (wire (pts (xy 206.375 59.055) (xy 210.185 59.055))
     (stroke (width 0) (type default) (color 0 0 0 0))
@@
     (stroke (width 0) (type default) (color 0 0 0 0))
   )
-  (wire (pts (xy 219.075 120.015) (xy 229.235 120.015))
+  (wire (pts (xy 219.075 120.015) (xy 226.695 120.015))
     (stroke (width 0) (type default) (color 0 0 0 0))
   )
@@
     (stroke (width 0) (type default) (color 0 0 0 0))
   )
+  (wire (pts (xy 134.62 53.34) (xy 138.43 53.34))
+    (stroke (width 0) (type default) (color 0 0 0 0))
+  )
   (wire (pts (xy 97.79 70.485) (xy 97.79 66.04))
     (stroke (width 0) (type default) (color 0 0 0 0))
@@
     (stroke (width 0) (type default) (color 0 0 0 0))
   )
+  (wire (pts (xy 250.19 120.015) (xy 254 120.015))
+    (stroke (width 0) (type default) (color 0 0 0 0))
+  )
   (wire (pts (xy 250.825 59.055) (xy 261.62 59.055))
     (stroke (width 0) (type default) (color 0 0 0 0))
@@
     (stroke (width 0) (type default) (color 0 0 0 0))
   )
-  (wire (pts (xy 132.08 53.34) (xy 138.43 53.34))
+  (wire (pts (xy 132.08 53.34) (xy 134.62 53.34))
     (stroke (width 0) (type default) (color 0 0 0 0))
   )
@@
     )
     (property "Datasheet" "" (id 3) (at 198.12 116.205 0)
+      (effects (font (size 1.27 1.27)) hide)
+    )
+    (pin "1")
+  )
+  (symbol (lib_id "Connector:TestPoint") (at 137.795 152.4 0) (unit 1)
+    (in_bom yes) (on_board yes) (fields_autoplaced)
+    (property "Reference" "TP18" (id 0) (at 140.335 147.8279 0)
+      (effects (font (size 1.27 1.27)) (justify left))
+    )
+    (property "Value" "TestPoint" (id 1) (at 140.335 150.3679 0)
+      (effects (font (size 1.27 1.27)) (justify left))
+    )
+    (property "Footprint" "" (id 2) (at 142.875 152.4 0)
+      (effects (font (size 1.27 1.27)) hide)
+    )
+    (property "Datasheet" "~" (id 3) (at 142.875 152.4 0)
+      (effects (font (size 1.27 1.27)) hide)
+    )
+    (pin "1")
+  )
+  (symbol (lib_id "Connector:TestPoint") (at 134.62 53.34 180) (unit 1)
+    (in_bom yes) (on_board yes) (fields_autoplaced)
+    (property "Reference" "TP17" (id 0) (at 136.525 55.3719 0)
+      (effects (font (size 1.27 1.27)) (justify right))
+    )
+    (property "Value" "TestPoint" (id 1) (at 136.525 57.9119 0)
+      (effects (font (size 1.27 1.27)) (justify right))
+    )
+    (property "Footprint" "" (id 2) (at 129.54 53.34 0)
+      (effects (font (size 1.27 1.27)) hide)
+    )
+    (property "Datasheet" "~" (id 3) (at 129.54 53.34 0)
       (effects (font (size 1.27 1.27)) hide)
     )
@@
     (pin "8")
   )
+  (symbol (lib_id "Connector:TestPoint") (at 250.19 120.015 0) (unit 1)
+    (in_bom yes) (on_board yes) (fields_autoplaced)
+    (property "Reference" "TP20" (id 0) (at 252.73 115.4429 0)
+      (effects (font (size 1.27 1.27)) (justify left))
+    )
+    (property "Value" "TestPoint" (id 1) (at 252.73 117.9829 0)
+      (effects (font (size 1.27 1.27)) (justify left))
+    )
+    (property "Footprint" "" (id 2) (at 255.27 120.015 0)
+      (effects (font (size 1.27 1.27)) hide)
+    )
+    (property "Datasheet" "~" (id 3) (at 255.27 120.015 0)
+      (effects (font (size 1.27 1.27)) hide)
+    )
+    (pin "1")
+  )
   (symbol (lib_id "Device:R") (at 196.215 48.26 90) (unit 1)
     (in_bom yes) (on_board yes)
@@
     (pin "1")
     (pin "2")
+  )
+  (symbol (lib_id "Connector:TestPoint") (at 276.86 50.165 180) (unit 1)
+    (in_bom yes) (on_board yes) (fields_autoplaced)
+    (property "Reference" "TP21" (id 0) (at 279.4 52.1969 0)
+      (effects (font (size 1.27 1.27)) (justify right))
+    )
+    (property "Value" "TestPoint" (id 1) (at 279.4 54.7369 0)
+      (effects (font (size 1.27 1.27)) (justify right))
+    )
+    (property "Footprint" "" (id 2) (at 271.78 50.165 0)
+      (effects (font (size 1.27 1.27)) hide)
+    )
+    (property "Datasheet" "~" (id 3) (at 271.78 50.165 0)
+      (effects (font (size 1.27 1.27)) hide)
+    )
+    (pin "1")
   )
   (symbol (lib_id "Device:R") (at 103.505 71.12 0) (unit 1)
@@
     (pin "2")
   )
+  (symbol (lib_id "Connector:TestPoint") (at 226.695 120.015 0) (unit 1)
+    (in_bom yes) (on_board yes) (fields_autoplaced)
+    (property "Reference" "TP19" (id 0) (at 229.235 115.4429 0)
+      (effects (font (size 1.27 1.27)) (justify left))
+    )
+    (property "Value" "TestPoint" (id 1) (at 229.235 117.9829 0)
+      (effects (font (size 1.27 1.27)) (justify left))
+    )
+    (property "Footprint" "" (id 2) (at 231.775 120.015 0)
+      (effects (font (size 1.27 1.27)) hide)
+    )
+    (property "Datasheet" "~" (id 3) (at 231.775 120.015 0)
+      (effects (font (size 1.27 1.27)) hide)
+    )
+    (pin "1")
+  )
+  (symbol (lib_id "Connector:TestPoint") (at 131.445 156.21 90) (unit 1)
+    (in_bom yes) (on_board yes) (fields_autoplaced)
+    (property "Reference" "TP16" (id 0) (at 128.143 149.86 90))
+    (property "Value" "TestPoint" (id 1) (at 128.143 152.4 90))
+    (property "Footprint" "" (id 2) (at 131.445 151.13 0)
+      (effects (font (size 1.27 1.27)) hide)
+    )
+    (property "Datasheet" "~" (id 3) (at 131.445 151.13 0)
+      (effects (font (size 1.27 1.27)) hide)
+    )
+    (pin "1")
+  )
   (symbol (lib_id "power:GND") (at 198.12 140.335 0) (unit 1)

Commit message: Working version
Parts:
- R28: value 1k -> 1.5k
- R30: value R -> 1k
- TP16, TP17, TP18, TP19, TP20, TP21: footprint (none) -> TestPoint:TestPoint_Pad_1.0x1.0mm
Changed lines of the file:
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@@
       (effects (font (size 1.27 1.27)) (justify left))
     )
-    (property "Footprint" "" (id 2) (at 142.875 152.4 0)
+    (property "Footprint" "TestPoint:TestPoint_Pad_1.0x1.0mm" (id 2) (at 142.875 152.4 0)
       (effects (font (size 1.27 1.27)) hide)
     )
@@
       (effects (font (size 1.27 1.27)) (justify right))
     )
-    (property "Footprint" "" (id 2) (at 129.54 53.34 0)
+    (property "Footprint" "TestPoint:TestPoint_Pad_1.0x1.0mm" (id 2) (at 129.54 53.34 0)
       (effects (font (size 1.27 1.27)) hide)
     )
@@
       (effects (font (size 1.27 1.27)) (justify left))
     )
-    (property "Footprint" "" (id 2) (at 255.27 120.015 0)
+    (property "Footprint" "TestPoint:TestPoint_Pad_1.0x1.0mm" (id 2) (at 255.27 120.015 0)
       (effects (font (size 1.27 1.27)) hide)
     )
@@
       (effects (font (size 1.27 1.27)) (justify right))
     )
-    (property "Footprint" "" (id 2) (at 271.78 50.165 0)
+    (property "Footprint" "TestPoint:TestPoint_Pad_1.0x1.0mm" (id 2) (at 271.78 50.165 0)
       (effects (font (size 1.27 1.27)) hide)
     )
@@
       (effects (font (size 1.27 1.27)) (justify left))
     )
-    (property "Value" "1k" (id 1) (at 209.55 135.2549 0)
+    (property "Value" "1.5k" (id 1) (at 209.55 135.2549 0)
       (effects (font (size 1.27 1.27)) (justify left))
     )
@@
       (effects (font (size 1.27 1.27)) (justify left))
     )
-    (property "Footprint" "" (id 2) (at 231.775 120.015 0)
+    (property "Footprint" "TestPoint:TestPoint_Pad_1.0x1.0mm" (id 2) (at 231.775 120.015 0)
       (effects (font (size 1.27 1.27)) hide)
     )
@@
     (property "Reference" "TP16" (id 0) (at 128.143 149.86 90))
     (property "Value" "TestPoint" (id 1) (at 128.143 152.4 90))
-    (property "Footprint" "" (id 2) (at 131.445 151.13 0)
+    (property "Footprint" "TestPoint:TestPoint_Pad_1.0x1.0mm" (id 2) (at 131.445 151.13 0)
       (effects (font (size 1.27 1.27)) hide)
     )
@@
       (effects (font (size 1.27 1.27)) (justify left))
     )
-    (property "Value" "R" (id 1) (at 220.98 125.7299 0)
-      (effects (font (size 1.27 1.27)) (justify left))
-    )
+    (property "Value" "1k" (id 1) (at 220.98 125.7299 0)
+      (effects (font (size 1.27 1.27)) (justify left))
+    )
