File: esc/3phases.kicad_sch (KiCad schematic)
At the start: 31 parts

Commit message: Finished layout
Parts:
- added R57, R58: 33, Resistor_SMD:R_0603_1608Metric, symbol Device:R
- C10, C11, C7: renamed from C?; value C -> 300p; footprint (none) -> Capacitor_SMD:C_0603_1608Metric
- C12, C13: renamed from C?; value C -> 100n; footprint (none) -> Capacitor_SMD:C_0603_1608Metric
- C8, C9: renamed from C?; footprint (none) -> Capacitor_SMD:C_0603_1608Metric
- R10, R11, R8, R9: renamed from R?; value R -> 100; footprint (none) -> Resistor_SMD:R_0603_1608Metric
- R12, R14, R20: renamed from R?; value R -> 8.2k; footprint (none) -> Resistor_SMD:R_0603_1608Metric
- R13, R15, R21: renamed from R?; value R -> 1k; footprint (none) -> Resistor_SMD:R_0603_1608Metric
- R16, R17, R18, R19: renamed from R?; value R -> 4.3k; footprint (none) -> Resistor_SMD:R_0603_1608Metric
- R2, R3, R4, R5, R6, R7: renamed from R?; value R -> 3m; footprint (none) -> Resistor_SMD:R_2512_6332Metric
- R22, R23: renamed from R?; value R -> 2.2k; footprint (none) -> Resistor_SMD:R_0603_1608Metric
- gave numbers to parts that had none: 2
Connections:
- net A_CURRENT_SENSE: now also R57.1; no longer R22.1, U2.1
- net B_CURRENT_SENSE: now also R58.1; no longer R23.1, U3.1
- net +3V3 renamed +3.3VA
- net GND renamed GNDA
- new net: R23.1, R58.2, U3.1
- new net: R22.1, R57.2, U2.1

Commit message: Finished design - first submission
Parts:
- added TP10, TP11, TP12, TP13, TP14, TP4, TP5, TP6, TP7, TP8, TP9: TestPoint, symbol Connector:TestPoint
Connections:
- net A_CURRENT_SENSE: now also TP13.1
- net A_HIN: now also TP4.1
- net A_VOLTAGE_SENSE: now also TP10.1
- net B_CURRENT_SENSE: now also TP14.1
- net B_HIN: now also TP6.1
- net B_VOLTAGE_SENSE: now also TP11.1
- net C_HIN: now also TP8.1
- net C_VOLTAGE_SENSE: now also TP12.1
- net ~{A_LIN}: now also TP5.1
- net ~{B_LIN}: now also TP7.1
- net ~{C_LIN}: now also TP9.1

Commit message: Working version
Parts:
- R10, R11, R8, R9: value 100 -> 120
- R16, R17, R18, R19: value 4.3k -> 6.6k
- R22, R23: value 2.2k -> 3.3k
- TP10, TP11, TP12, TP13, TP14, TP4, TP5, TP6, TP7, TP8, TP9: footprint (none) -> TestPoint:TestPoint_Pad_1.0x1.0mm
Changed lines of the file:
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@@
       (effects (font (size 1.27 1.27)) (justify left))
     )
-    (property "Footprint" "" (id 2) (at 325.755 208.28 0)
+    (property "Footprint" "TestPoint:TestPoint_Pad_1.0x1.0mm" (id 2) (at 325.755 208.28 0)
       (effects (font (size 1.27 1.27)) hide)
     )
@@
       (effects (font (size 1.27 1.27)) (justify right))
     )
-    (property "Value" "4.3k" (id 1) (at 274.32 147.3199 0)
+    (property "Value" "6.6k" (id 1) (at 274.32 147.3199 0)
       (effects (font (size 1.27 1.27)) (justify right))
     )
@@
   )
   (symbol (lib_id "Connector:TestPoint") (at 97.79 99.695 0) (unit 1)
-    (in_bom yes) (on_board yes) (fields_autoplaced)
-    (property "Reference" "TP8" (id 0) (at 100.33 95.1229 0)
+    (in_bom yes) (on_board yes)
+    (property "Reference" "TP8" (id 0) (at 97.79 94.615 90)
       (effects (font (size 1.27 1.27)) (justify left))
     )
@@
       (effects (font (size 1.27 1.27)) (justify left))
     )
-    (property "Footprint" "" (id 2) (at 102.87 99.695 0)
+    (property "Footprint" "TestPoint:TestPoint_Pad_1.0x1.0mm" (id 2) (at 102.87 99.695 0)
       (effects (font (size 1.27 1.27)) hide)
     )
@@
   )
   (symbol (lib_id "Connector:TestPoint") (at 90.17 99.695 0) (unit 1)
-    (in_bom yes) (on_board yes) (fields_autoplaced)
-    (property "Reference" "TP4" (id 0) (at 92.71 95.1229 0)
+    (in_bom yes) (on_board yes)
+    (property "Reference" "TP4" (id 0) (at 90.17 94.615 90)
       (effects (font (size 1.27 1.27)) (justify left))
     )
@@
       (effects (font (size 1.27 1.27)) (justify left))
     )
-    (property "Footprint" "" (id 2) (at 95.25 99.695 0)
+    (property "Footprint" "TestPoint:TestPoint_Pad_1.0x1.0mm" (id 2) (at 95.25 99.695 0)
       (effects (font (size 1.27 1.27)) hide)
     )
@@
       (effects (font (size 1.27 1.27)) (justify left))
     )
-    (property "Footprint" "" (id 2) (at 325.755 159.385 0)
+    (property "Footprint" "TestPoint:TestPoint_Pad_1.0x1.0mm" (id 2) (at 325.755 159.385 0)
       (effects (font (size 1.27 1.27)) hide)
     )
@@
       (effects (font (size 1.27 1.27)) (justify left))
     )
-    (property "Footprint" "" (id 2) (at 318.135 109.855 0)
+    (property "Footprint" "TestPoint:TestPoint_Pad_1.0x1.0mm" (id 2) (at 318.135 109.855 0)
       (effects (font (size 1.27 1.27)) hide)
     )
@@
     (in_bom yes) (on_board yes)
     (property "Reference" "R23" (id 0) (at 297.815 221.615 90))
-    (property "Value" "2.2k" (id 1) (at 297.815 219.71 90))
+    (property "Value" "3.3k" (id 1) (at 297.815 219.71 90))
     (property "Footprint" "Resistor_SMD:R_0603_1608Metric" (id 2) (at 297.815 218.948 90)
       (effects (font (size 1.27 1.27)) hide)
@@
       (effects (font (size 1.27 1.27)) (justify right))
     )
-    (property "Value" "4.3k" (id 1) (at 274.32 168.9099 0)
+    (property "Value" "6.6k" (id 1) (at 274.32 168.9099 0)
       (effects (font (size 1.27 1.27)) (justify right))
     )
@@
       (effects (font (size 1.27 1.27)) (justify left))
     )
-    (property "Footprint" "" (id 2) (at 314.325 109.855 0)
+    (property "Footprint" "TestPoint:TestPoint_Pad_1.0x1.0mm" (id 2) (at 314.325 109.855 0)
       (effects (font (size 1.27 1.27)) hide)
     )
@@
     (in_bom yes) (on_board yes)
     (property "Reference" "R22" (id 0) (at 297.815 172.72 90))
-    (property "Value" "2.2k" (id 1) (at 297.815 170.815 90))
+    (property "Value" "3.3k" (id 1) (at 297.815 170.815 90))
     (property "Footprint" "Resistor_SMD:R_0603_1608Metric" (id 2) (at 297.815 170.053 90)
       (effects (font (size 1.27 1.27)) hide)
@@
       (effects (font (size 1.27 1.27)) (justify right))
     )
-    (property "Value" "4.3k" (id 1) (at 274.32 217.8049 0)
+    (property "Value" "6.6k" (id 1) (at 274.32 217.8049 0)
       (effects (font (size 1.27 1.27)) (justify right))
     )
@@
   )
   (symbol (lib_id "Connector:TestPoint") (at 95.885 99.695 0) (unit 1)
-    (in_bom yes) (on_board yes) (fields_autoplaced)
-    (property "Reference" "TP7" (id 0) (at 98.425 95.1229 0)
+    (in_bom yes) (on_board yes)
+    (property "Reference" "TP7" (id 0) (at 95.885 94.615 90)
       (effects (font (size 1.27 1.27)) (justify left))
     )
@@
       (effects (font (size 1.27 1.27)) (justify left))
     )
-    (property "Footprint" "" (id 2) (at 100.965 99.695 0)
+    (property "Footprint" "TestPoint:TestPoint_Pad_1.0x1.0mm" (id 2) (at 100.965 99.695 0)
       (effects (font (size 1.27 1.27)) hide)
     )
@@
       (effects (font (size 1.27 1.27)) (justify left))
     )
-    (property "Footprint" "" (id 2) (at 316.23 109.855 0)
+    (property "Footprint" "TestPoint:TestPoint_Pad_1.0x1.0mm" (id 2) (at 316.23 109.855 0)
       (effects (font (size 1.27 1.27)) hide)
     )
@@
       (effects (font (size 1.27 1.27)) (justify right))
     )
-    (property "Value" "4.3k" (id 1) (at 274.32 196.2149 0)
+    (property "Value" "6.6k" (id 1) (at 274.32 196.2149 0)
       (effects (font (size 1.27 1.27)) (justify right))
     )
@@
     (in_bom yes) (on_board yes) (fields_autoplaced)
     (property "Reference" "R8" (id 0) (at 248.92 151.13 90))
-    (property "Value" "100" (id 1) (at 248.92 153.67 90))
+    (property "Value" "120" (id 1) (at 248.92 153.67 90))
     (property "Footprint" "Resistor_SMD:R_0603_1608Metric" (id 2) (at 248.92 158.623 90)
       (effects (font (size 1.27 1.27)) hide)
@@
     (in_bom yes) (on_board yes) (fields_autoplaced)
     (property "Reference" "R9" (id 0) (at 248.92 156.21 90))
-    (property "Value" "100" (id 1) (at 248.92 158.75 90))
+    (property "Value" "120" (id 1) (at 248.92 158.75 90))
     (property "Footprint" "Resistor_SMD:R_0603_1608Metric" (id 2) (at 248.92 163.703 90)
       (effects (font (size 1.27 1.27)) hide)
@@
   )
   (symbol (lib_id "Connector:TestPoint") (at 92.075 99.695 0) (unit 1)
-    (in_bom yes) (on_board yes) (fields_autoplaced)
-    (property "Reference" "TP5" (id 0) (at 94.615 95.1229 0)
+    (in_bom yes) (on_board yes)
+    (property "Reference" "TP5" (id 0) (at 92.075 94.615 90)
       (effects (font (size 1.27 1.27)) (justify left))
     )
@@
       (effects (font (size 1.27 1.27)) (justify left))
     )
-    (property "Footprint" "" (id 2) (at 97.155 99.695 0)
+    (property "Footprint" "TestPoint:TestPoint_Pad_1.0x1.0mm" (id 2) (at 97.155 99.695 0)
       (effects (font (size 1.27 1.27)) hide)
     )
@@
     (in_bom yes) (on_board yes) (fields_autoplaced)
     (property "Reference" "R10" (id 0) (at 248.92 199.39 90))
-    (property "Value" "100" (id 1) (at 248.92 201.93 90))
+    (property "Value" "120" (id 1) (at 248.92 201.93 90))
     (property "Footprint" "Resistor_SMD:R_0603_1608Metric" (id 2) (at 248.92 207.518 90)
       (effects (font (size 1.27 1.27)) hide)
@@
     (in_bom yes) (on_board yes) (fields_autoplaced)
     (property "Reference" "R11" (id 0) (at 248.92 204.47 90))
-    (property "Value" "100" (id 1) (at 248.92 207.01 90))
+    (property "Value" "120" (id 1) (at 248.92 207.01 90))
     (property "Footprint" "Resistor_SMD:R_0603_1608Metric" (id 2) (at 248.92 212.598 90)
       (effects (font (size 1.27 1.27)) hide)
@@
   )
   (symbol (lib_id "Connector:TestPoint") (at 93.98 99.695 0) (unit 1)
-    (in_bom yes) (on_board yes) (fields_autoplaced)
-    (property "Reference" "TP6" (id 0) (at 96.52 95.1229 0)
+    (in_bom yes) (on_board yes)
+    (property "Reference" "TP6" (id 0) (at 93.98 94.615 90)
       (effects (font (size 1.27 1.27)) (justify left))
     )
@@
       (effects (font (size 1.27 1.27)) (justify left))
     )
-    (property "Footprint" "" (id 2) (at 99.06 99.695 0)
+    (property "Footprint" "TestPoint:TestPoint_Pad_1.0x1.0mm" (id 2) (at 99.06 99.695 0)
       (effects (font (size 1.27 1.27)) hide)
     )
@@
   )
   (symbol (lib_id "Connector:TestPoint") (at 99.695 99.695 0) (unit 1)
-    (in_bom yes) (on_board yes) (fields_autoplaced)
-    (property "Reference" "TP9" (id 0) (at 102.235 95.1229 0)
+    (in_bom yes) (on_board yes)
+    (property "Reference" "TP9" (id 0) (at 99.695 94.615 90)
       (effects (font (size 1.27 1.27)) (justify left))
     )
@@
       (effects (font (size 1.27 1.27)) (justify left))
     )
-    (property "Footprint" "" (id 2) (at 104.775 99.695 0)
-      (effects (font (size 1.27 1.27)) hide)
-    )
+    (property "Footprint" "TestPoint:TestPoint_Pad_1.0x1.0mm" (id 2) (at 104.775 99.695 0)
+      (effects (font (size 1.27 1.27)) hide)
+    )

Commit message: Some stuff
Parts:
- removed C10, C11, C7: 300p, Capacitor_SMD:C_0603_1608Metric, symbol Device:C
- removed R12, R14, R20: 8.2k, Resistor_SMD:R_0603_1608Metric, symbol Device:R
- removed R13, R15, R21: 1k, Resistor_SMD:R_0603_1608Metric, symbol Device:R
- removed TP10, TP11, TP12, TP13, TP14: TestPoint, TestPoint:TestPoint_Pad_1.0x1.0mm, symbol Connector:TestPoint
- added J10, J11, J84, J86, J90, J91: Conn_01x01, Library:SmallPin, symbol Connector_Generic:Conn_01x01
- added J8, J85, J87, J88, J89, J9: Conn_01x01, Library:SmallPad, symbol Connector_Generic:Conn_01x01
- added R30, R31, R32, R59: 3.3k, Resistor_SMD:R_0603_1608Metric, symbol Device:R
- C8, C9: value C -> 1n
- R16, R17, R18, R19: value 6.6k -> 3.3k
Connections:
- net +3.3VA: now also J84.1 (Pin_1), J86.1 (Pin_1); no longer C12.1, C13.1, R16.2, R18.2, U2.5 (V+), U3.5 (V+)
- net A_CURRENT_SENSE: now also J10.1 (Pin_1); no longer R57.1
- net B_CURRENT_SENSE: now also J11.1 (Pin_1); no longer R58.1
- net GNDA: now also J90.1 (Pin_1), J91.1 (Pin_1); no longer C12.2, C13.2, C8.2, C9.2, R17.1, R19.1, U2.2 (V-), U3.2 (V-)
- net at R11.1, R23.2, U3.4 (-): now also C9.2
- net at R22.2, R9.1, U2.4 (-): now also C8.2
- new net: C12.2, J88.1 (Pin_1), R31.1, U2.2 (V-)
- new net: R17.1, R31.2
- new net: C13.1, J85.1 (Pin_1), R32.1, U3.5 (V+)
- new net: R16.2, R30.1
- new net: C12.1, J87.1 (Pin_1), R30.2, U2.5 (V+)
- new net: C13.2, J89.1 (Pin_1), R59.2, U3.2 (V-)
- new net: R19.1, R59.1
- new net: J8.1 (Pin_1), R57.1
- new net: J9.1 (Pin_1), R58.1
- new net: R18.2, R32.2
Other:
- note added: "Time constant = 240ns"
- moved on the sheet: C12, C13, C8, C9, R10, R11, R16, R17, R18, R19, R22, R23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

Commit message: Pretty much finished new design
Parts:
- removed J88, J89: Conn_01x01, Library:SmallPad, symbol Connector_Generic:Conn_01x01
- removed J90, J91: Conn_01x01, Library:SmallPin, symbol Connector_Generic:Conn_01x01
- removed TP4, TP5, TP6, TP7, TP8, TP9: TestPoint, TestPoint:TestPoint_Pad_1.0x1.0mm, symbol Connector:TestPoint
- J10, J11: footprint Library:SmallPin -> Library:SmallPad
- J85, J87: footprint Library:SmallPad -> Library:SmallPin
Connections:
- net +3.3VA: now also C12.1, C13.1, R30.2, R32.1, U2.5 (V+), U3.5 (V+); no longer J84.1 (Pin_1), J86.1 (Pin_1)
- net A_CURRENT_SENSE: now also R57.1; no longer J10.1 (Pin_1)
- net B_CURRENT_SENSE: now also R58.1; no longer J11.1 (Pin_1)
- net GNDA: now also C12.2, C13.2, R31.1, R59.2, U2.2 (V-), U3.2 (V-)
- net POWER-: now also J11.1 (Pin_1), J9.1 (Pin_1); no longer R11.2, R9.2
- net Phase A/BRIDGE_LOW: now also J8.1 (Pin_1); no longer R8.2
- net Phase B/BRIDGE_LOW: now also J10.1 (Pin_1); no longer R10.2
- new net: J84.1 (Pin_1), R8.2
- new net: J85.1 (Pin_1), R9.2
- new net: J86.1 (Pin_1), R10.2
- new net: J87.1 (Pin_1), R11.2
