File: esc/esc.kicad_sch (KiCad schematic)
At the start: 14 parts, among them J1 Conn_01x02, J2 Conn_01x03, J3 Conn_01x05, J4 Conn_01x05, J5 Conn_01x04, SW1 SW_SPDT, U1 dsPIC33CK64MC103

Commit message: Finished design - first submission
Parts:
- added TP3: TestPoint, symbol Connector:TestPoint
Connections:
- net LV_SUPPLY: now also TP3.1
Changed lines of the file:
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@@
   (junction (at 61.595 73.025) (diameter 0) (color 0 0 0 0)
+  )
+  (junction (at 96.52 45.085) (diameter 0) (color 0 0 0 0)
   )
   (junction (at 66.04 41.91) (diameter 0) (color 0 0 0 0)
@@
     (stroke (width 0) (type default) (color 0 0 0 0))
   )
+  (wire (pts (xy 96.52 45.085) (xy 98.425 45.085))
+    (stroke (width 0) (type default) (color 0 0 0 0))
+  )
   (wire (pts (xy 240.03 124.46) (xy 252.73 124.46))
     (stroke (width 1) (type default) (color 0 0 0 0))
@@
     (stroke (width 0) (type default) (color 0 0 0 0))
   )
-  (wire (pts (xy 93.98 45.085) (xy 98.425 45.085))
+  (wire (pts (xy 93.98 45.085) (xy 96.52 45.085))
     (stroke (width 0) (type default) (color 0 0 0 0))
   )
@@
     (stroke (width 0) (type default) (color 0 0 0 0))
   )
+  (wire (pts (xy 29.21 27.94) (xy 49.53 27.94))
+    (stroke (width 1) (type default) (color 0 0 0 0))
+  )
   (wire (pts (xy 108.585 42.545) (xy 111.125 42.545))
     (stroke (width 0) (type default) (color 0 0 0 0))
@@
   (wire (pts (xy 91.44 171.45) (xy 98.425 171.45))
     (stroke (width 0) (type default) (color 0 0 0 0))
-  )
-  (wire (pts (xy 29.21 27.94) (xy 49.53 27.94))
-    (stroke (width 1) (type default) (color 0 0 0 0))
   )
   (wire (pts (xy 49.53 60.325) (xy 49.53 62.23))
@@
     (pin "1")
     (pin "2")
+  )
+  (symbol (lib_id "Connector:TestPoint") (at 96.52 45.085 180) (unit 1)
+    (in_bom yes) (on_board yes) (fields_autoplaced)
+    (property "Reference" "TP3" (id 0) (at 99.06 47.1169 0)
+      (effects (font (size 1.27 1.27)) (justify right))
+    )
+    (property "Value" "TestPoint" (id 1) (at 99.06 49.6569 0)
+      (effects (font (size 1.27 1.27)) (justify right))
+    )
+    (property "Footprint" "" (id 2) (at 91.44 45.085 0)
+      (effects (font (size 1.27 1.27)) hide)
+    )
+    (property "Datasheet" "~" (id 3) (at 91.44 45.085 0)
+      (effects (font (size 1.27 1.27)) hide)
+    )
+    (pin "1")
   )
   (symbol (lib_id "power:+3.3VA") (at 69.215 66.675 0) (unit 1)
@@
       (reference "SW3") (unit 1) (value "SW_SPDT") (footprint "Connector_PinHeader_2.54mm:PinHeader_1x03_P2.54mm_Vertical")
     )
+    (path "/4972b020-4774-4db1-ad0e-3671087ece28"
+      (reference "TP3") (unit 1) (value "TestPoint") (footprint "TestPoint:TestPoint_Pad_1.0x1.0mm")
+    )
+    (path "/411d4270-c66c-4318-b7fb-1470d34862b8/38ecdee2-49d2-4ec9-b664-af6f843820c3"
+      (reference "TP4") (unit 1) (value "TestPoint") (footprint "TestPoint:TestPoint_Pad_1.0x1.0mm")
+    )
+    (path "/411d4270-c66c-4318-b7fb-1470d34862b8/d0e02675-d3e1-4170-b833-5effca6086fa"
+      (reference "TP5") (unit 1) (value "TestPoint") (footprint "TestPoint:TestPoint_Pad_1.0x1.0mm")
+    )
+    (path "/411d4270-c66c-4318-b7fb-1470d34862b8/e35fb9d5-1b2a-44be-a071-87642b610268"
+      (reference "TP6") (unit 1) (value "TestPoint") (footprint "TestPoint:TestPoint_Pad_1.0x1.0mm")
+    )
+    (path "/411d4270-c66c-4318-b7fb-1470d34862b8/7bbc94c5-94f5-416f-b33b-c202ad6acb39"
+      (reference "TP7") (unit 1) (value "TestPoint") (footprint "TestPoint:TestPoint_Pad_1.0x1.0mm")
+    )
+    (path "/411d4270-c66c-4318-b7fb-1470d34862b8/38af322a-aa37-4376-afd0-d8d67257831b"
+      (reference "TP8") (unit 1) (value "TestPoint") (footprint "TestPoint:TestPoint_Pad_1.0x1.0mm")
+    )
+    (path "/411d4270-c66c-4318-b7fb-1470d34862b8/f17d6d70-35ce-4ad3-a2be-a3b709d2b53c"
+      (reference "TP9") (unit 1) (value "TestPoint") (footprint "TestPoint:TestPoint_Pad_1.0x1.0mm")
+    )
+    (path "/411d4270-c66c-4318-b7fb-1470d34862b8/5c9d36e8-7f55-4c5c-8951-f68307312c81"
+      (reference "TP10") (unit 1) (value "TestPoint") (footprint "TestPoint:TestPoint_Pad_1.0x1.0mm")
+    )
+    (path "/411d4270-c66c-4318-b7fb-1470d34862b8/9d81e19f-6b7d-4d77-878e-735d079f25e6"
+      (reference "TP11") (unit 1) (value "TestPoint") (footprint "TestPoint:TestPoint_Pad_1.0x1.0mm")
+    )
+    (path "/411d4270-c66c-4318-b7fb-1470d34862b8/44779a4f-680b-4951-9c1a-6ef76154a6bc"
+      (reference "TP12") (unit 1) (value "TestPoint") (footprint "TestPoint:TestPoint_Pad_1.0x1.0mm")
+    )
+    (path "/411d4270-c66c-4318-b7fb-1470d34862b8/3adb0d71-8748-4459-9712-1a567459170f"
+      (reference "TP13") (unit 1) (value "TestPoint") (footprint "TestPoint:TestPoint_Pad_1.0x1.0mm")
+    )
+    (path "/411d4270-c66c-4318-b7fb-1470d34862b8/196258df-c159-4719-a6a4-7b7c9d2700d0"
+      (reference "TP14") (unit 1) (value "TestPoint") (footprint "TestPoint:TestPoint_Pad_1.0x1.0mm")
+    )
+    (path "/3efd3b84-f628-4891-a9d4-352b6e1fc0c5/c4396c99-ca0c-464b-a785-d60b54b14e25"
+      (reference "TP16") (unit 1) (value "TestPoint") (footprint "TestPoint:TestPoint_Pad_1.0x1.0mm")
+    )
+    (path "/3efd3b84-f628-4891-a9d4-352b6e1fc0c5/231930a8-5cea-46ad-ad9f-0d12ecb4d662"
+      (reference "TP17") (unit 1) (value "TestPoint") (footprint "TestPoint:TestPoint_Pad_1.0x1.0mm")
+    )
+    (path "/3efd3b84-f628-4891-a9d4-352b6e1fc0c5/21c68380-a80d-4471-9923-d543922a628d"
+      (reference "TP18") (unit 1) (value "TestPoint") (footprint "TestPoint:TestPoint_Pad_1.0x1.0mm")
+    )
+    (path "/3efd3b84-f628-4891-a9d4-352b6e1fc0c5/c3f2f465-fbc0-4d61-8ca9-85d5a5ebffec"
+      (reference "TP19") (unit 1) (value "TestPoint") (footprint "TestPoint:TestPoint_Pad_1.0x1.0mm")
+    )
+    (path "/3efd3b84-f628-4891-a9d4-352b6e1fc0c5/324337f4-10dd-438f-8da5-d095f0b25a4e"
+      (reference "TP20") (unit 1) (value "TestPoint") (footprint "TestPoint:TestPoint_Pad_1.0x1.0mm")
+    )
+    (path "/3efd3b84-f628-4891-a9d4-352b6e1fc0c5/51469661-4062-44ed-b4f1-f2328dbe72e1"
+      (reference "TP21") (unit 1) (value "TestPoint") (footprint "TestPoint:TestPoint_Pad_1.0x1.0mm")
+    )
     (path "/76cd2633-5bc8-425f-b0a9-11ce11dc8546"

Commit message: Working version
Parts:
- TP3: footprint (none) -> TestPoint:TestPoint_Pad_1.0x1.0mm
Other:
- note added: "3V3 on hall connector"
Changed lines of the file:
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@@
     (stroke (width 1) (type default) (color 0 0 0 0))
+  )
+  (text "3V3 on hall connector" (at 153.67 167.005 0)
+    (effects (font (size 1.27 1.27) italic) (justify left bottom))
   )
   (label "QEI_A{slash}HALL_A{slash}GPIO0" (at 145.415 173.99 180)
@@
       (effects (font (size 1.27 1.27)) (justify right))
     )
-    (property "Footprint" "" (id 2) (at 91.44 45.085 0)
+    (property "Footprint" "TestPoint:TestPoint_Pad_1.0x1.0mm" (id 2) (at 91.44 45.085 0)
       (effects (font (size 1.27 1.27)) hide)
     )
@@
     )
     (path "/411d4270-c66c-4318-b7fb-1470d34862b8/c5b67bdf-a002-474d-88d6-cf5ee755877e"
-      (reference "R8") (unit 1) (value "100") (footprint "Resistor_SMD:R_0603_1608Metric")
+      (reference "R8") (unit 1) (value "120") (footprint "Resistor_SMD:R_0603_1608Metric")
     )
     (path "/411d4270-c66c-4318-b7fb-1470d34862b8/cd2ace63-3850-4a00-8c93-26b39bc8ddd0"
-      (reference "R9") (unit 1) (value "100") (footprint "Resistor_SMD:R_0603_1608Metric")
+      (reference "R9") (unit 1) (value "120") (footprint "Resistor_SMD:R_0603_1608Metric")
     )
     (path "/411d4270-c66c-4318-b7fb-1470d34862b8/da3d6292-ba43-40b5-921c-1d6babfe980d"
-      (reference "R10") (unit 1) (value "100") (footprint "Resistor_SMD:R_0603_1608Metric")
+      (reference "R10") (unit 1) (value "120") (footprint "Resistor_SMD:R_0603_1608Metric")
     )
     (path "/411d4270-c66c-4318-b7fb-1470d34862b8/dcd1818f-2bdc-4713-bb2d-08cccd6ac4ca"
-      (reference "R11") (unit 1) (value "100") (footprint "Resistor_SMD:R_0603_1608Metric")
+      (reference "R11") (unit 1) (value "120") (footprint "Resistor_SMD:R_0603_1608Metric")
     )
     (path "/411d4270-c66c-4318-b7fb-1470d34862b8/c0b51b6d-fc93-45f0-bc02-610f3d8d701c"
@@
     )
     (path "/411d4270-c66c-4318-b7fb-1470d34862b8/2ec22a05-7bee-4939-87f5-78f979e48993"
-      (reference "R16") (unit 1) (value "4.3k") (footprint "Resistor_SMD:R_0603_1608Metric")
+      (reference "R16") (unit 1) (value "6.6k") (footprint "Resistor_SMD:R_0603_1608Metric")
     )
     (path "/411d4270-c66c-4318-b7fb-1470d34862b8/59957bb2-dec9-4d1c-914e-9452f1c8f626"
-      (reference "R17") (unit 1) (value "4.3k") (footprint "Resistor_SMD:R_0603_1608Metric")
+      (reference "R17") (unit 1) (value "6.6k") (footprint "Resistor_SMD:R_0603_1608Metric")
     )
     (path "/411d4270-c66c-4318-b7fb-1470d34862b8/bcf62530-a923-4fba-b51b-7ba9f15fc47e"
-      (reference "R18") (unit 1) (value "4.3k") (footprint "Resistor_SMD:R_0603_1608Metric")
+      (reference "R18") (unit 1) (value "6.6k") (footprint "Resistor_SMD:R_0603_1608Metric")
     )
     (path "/411d4270-c66c-4318-b7fb-1470d34862b8/6fb826ef-0a0e-460d-918f-3433d5f3b960"
-      (reference "R19") (unit 1) (value "4.3k") (footprint "Resistor_SMD:R_0603_1608Metric")
+      (reference "R19") (unit 1) (value "6.6k") (footprint "Resistor_SMD:R_0603_1608Metric")
     )
     (path "/411d4270-c66c-4318-b7fb-1470d34862b8/f9a1f94a-1d2a-46f3-8304-e118d957fe50"
@@
     )
     (path "/411d4270-c66c-4318-b7fb-1470d34862b8/65181d3c-d299-4f9b-92af-e4388f5e5c0f"
-      (reference "R22") (unit 1) (value "2.2k") (footprint "Resistor_SMD:R_0603_1608Metric")
+      (reference "R22") (unit 1) (value "3.3k") (footprint "Resistor_SMD:R_0603_1608Metric")
     )
     (path "/411d4270-c66c-4318-b7fb-1470d34862b8/480da44a-f58e-44a2-a632-efdaf5587042"
-      (reference "R23") (unit 1) (value "2.2k") (footprint "Resistor_SMD:R_0603_1608Metric")
+      (reference "R23") (unit 1) (value "3.3k") (footprint "Resistor_SMD:R_0603_1608Metric")
     )
     (path "/3efd3b84-f628-4891-a9d4-352b6e1fc0c5/1d05dc79-dda4-4316-873d-d31fd1c2042b"
@@
     )
     (path "/3efd3b84-f628-4891-a9d4-352b6e1fc0c5/73012d62-09f7-4e13-998e-800cf36a3c2b"
-      (reference "R28") (unit 1) (value "1k") (footprint "Resistor_SMD:R_0603_1608Metric")
+      (reference "R28") (unit 1) (value "1.5k") (footprint "Resistor_SMD:R_0603_1608Metric")
     )
     (path "/3efd3b84-f628-4891-a9d4-352b6e1fc0c5/9ba406a6-8a27-446b-ae89-6a25c468570c"
@@
     )
     (path "/3efd3b84-f628-4891-a9d4-352b6e1fc0c5/f5b1add7-59e1-4f0a-a90f-7cc92c959d72"
-      (reference "R30") (unit 1) (value "R") (footprint "Resistor_SMD:R_0603_1608Metric")
+      (reference "R30") (unit 1) (value "1k") (footprint "Resistor_SMD:R_0603_1608Metric")
     )
     (path "/3efd3b84-f628-4891-a9d4-352b6e1fc0c5/3c7b59f8-157a-48d0-bcbd-1b5daab963d2"

Commit message: Some stuff
Parts:
- removed J5: Conn_01x04, Connector_PinHeader_2.54mm:PinHeader_1x04_P2.54mm_Vertical, symbol Connector_Generic:Conn_01x04
- removed SW1: SW_SPDT, Connector_PinHeader_2.54mm:PinHeader_1x03_P2.54mm_Vertical, symbol Switch:SW_SPDT
- removed TP3: TestPoint, TestPoint:TestPoint_Pad_1.0x1.0mm, symbol Connector:TestPoint
- added C10, C11, C14, C19, C20, C21, C7: 1n, Capacitor_SMD:C_0603_1608Metric, symbol Device:C
- added C15, C16, C17, C22: 10u, Capacitor_SMD:C_0805_2012Metric, symbol Device:C
- added C18: 1u, Capacitor_SMD:C_0603_1608Metric, symbol Device:C
- added J5: Conn_01x03, symbol Connector_Generic:Conn_01x03
- added J6: Conn_01x04, symbol Connector_Generic:Conn_01x04
- added J7: Conn_01x05, Connector_PinHeader_2.54mm:PinHeader_1x05_P2.54mm_Horizontal, symbol Connector_Generic:Conn_01x05
- added NT1: NetTie_2, footprints:Nettie2, symbol Device:NetTie_2
- added R12, R13, R14, R15: 330, Resistor_SMD:R_0603_1608Metric, symbol Device:R
- added R20: 1.5k, Resistor_SMD:R_0603_1608Metric, symbol Device:R
- added R21, R24, R25, R26, R27, R28, R29: 1k, Resistor_SMD:R_0603_1608Metric, symbol Device:R
- added TP1, TP2: TestPoint, TestPoint:TestPoint_Pad_1.0x1.0mm, symbol Connector:TestPoint
- added U4: AP1117-ADJ, Package_TO_SOT_SMD:SOT-223-3_TabPin2, symbol Regulator_Linear:AP1117-ADJ
- J4: now left out of the parts list
Connections:
- net +12V: now also J5.1 (Pin_1)
- net +3.3VA: now also C17.1, C18.1, NT1.2, TP2.1
- net +3V3: now also C16.1, C22.1, J7.1 (Pin_1), NT1.1, R21.1, R27.1, R28.1, R29.1, TP1.1, U4.2 (VO)
- net GND: now also C10.2, C11.2, C14.2, C15.2, C16.2, C19.2, C20.2, C21.2, C22.2, C7.2, J5.3 (Pin_3), J7.5 (Pin_5), R20.2
- net GNDA: now also C17.2, C18.2
- net HOME/HALL_C/GPIO2: now also U1.30 (RP53/RC5), C21.1, R26.1; no longer U1.16 (AN15/IBIAS2/RP51/RC3)
- net QEI_A/HALL_A/GPIO0: now also U1.16 (AN15/IBIAS2/RP51/RC3), C19.1, R24.1; no longer U1.29 (RP52/RC4)
- net QEI_B/HALL_B/GPIO1: now also U1.29 (RP52/RC4), C20.1, R25.1; no longer U1.30 (RP53/RC5)
- net GPIO0: now reaches U1.17 (OSCI/CLKI/AN5/RP32/RB0)
- net GPIO0: now also C7.1, R12.2
- net GPIO1: now reaches U1.18 (OSCO/CLKO/AN6/RP33/RB1)
- net GPIO1: now also C10.1, R13.2
- net GPIO2: now reaches U1.19 (OA2OUT/AN1/AN7/CMP1D/RP34/INT0/RB2)
- net GPIO2: now also C11.1, R14.2
- net GPIO3: now reaches U1.20 (PGD2/OA2IN-/AN8/RP35/RB3)
- net GPIO3: now also C14.1, R15.2
- net Phases/A_VOLTAGE_SENSE: no longer names the net of U1.8 (DACOUT/AN3/CMP1C/RA3)
- net Phases/B_VOLTAGE_SENSE: no longer names the net of U1.9 (OA3OUT/AN4/IBIAS3/RA4)
- new net: J6.1 (Pin_1), R12.1
- new net: J6.2 (Pin_2), R13.1
- new net: J6.3 (Pin_3), R14.1
- new net: J6.4 (Pin_4), R15.1
- new net: J7.2 (Pin_2), R24.2, R27.2
- new net: J7.4 (Pin_4), R26.2, R29.2
- new net: J7.3 (Pin_3), R25.2, R28.2
- new net: R20.1, R21.2, U4.1 (ADJ)
- new net +5V: C15.1, J5.2 (Pin_2), U4.3 (VI)
- no-connect marks 8 -> 3
Other:
- removed sheet Supplies
- sheet Phases ports: added none; removed A_VOLTAGE_SENSE, B_VOLTAGE_SENSE
- note added: "3V3 supply"
- note added: "Control board"
- note added: "Control board input side connections"
- note added: "Control board output side connections"
- note added: "Control board power"
- note added: "GPIO"
- note added: "Power board"
- note added: "Power board input connections"
- note added: "Power board output connections"
- note added: "SPI comms"
- note removed: "3V3 on hall connector"
- moved on the sheet: C1, C2, C3, C4, C5, C6, J1, J2, J3, J4, R1, U1

Commit message: Pretty much finished new design
Parts:
- removed C10, C11, C14, C7: 1n, Capacitor_SMD:C_0603_1608Metric, symbol Device:C
- removed C18: 1u, Capacitor_SMD:C_0603_1608Metric, symbol Device:C
- removed C2, C5: 470u, footprints:HorizontalCap_10x16_P5, symbol Device:C_Polarized
- removed J5: Conn_01x03, symbol Connector_Generic:Conn_01x03
- removed NT1: NetTie_2, footprints:Nettie2, symbol Device:NetTie_2
- removed R12, R13, R14, R15: 330, Resistor_SMD:R_0603_1608Metric, symbol Device:R
- removed TP1, TP2: TestPoint, TestPoint:TestPoint_Pad_1.0x1.0mm, symbol Connector:TestPoint
- added J88: Conn_01x01, Library:SmallPad, symbol Connector_Generic:Conn_01x01
- added J89: Conn_01x01, Library:SmallPin, symbol Connector_Generic:Conn_01x01
- added R60, R61: 0R, Resistor_SMD:R_0603_1608Metric, symbol Device:R
- J3: footprint Connector_PinHeader_2.54mm:PinHeader_1x05_P2.54mm_Vertical -> footprints:ProgConnector
- J4: footprint Connector_PinHeader_2.54mm:PinHeader_1x05_P2.54mm_Vertical -> footprints:EdgeConnector_5; now in the parts list
- J6: footprint (none) -> footprints:EdgeConnector_4; now in the parts list
Connections:
- net +12V: now also J4.5 (Pin_5)
- net +3.3VA: now also R60.2
- net +3V3: now also R60.1
- net +5V: now also J4.4 (Pin_4)
- net GND: now also J4.1 (Pin_1), J89.1 (Pin_1), R61.1; no longer J4.5 (Pin_5)
- net GNDA: now also R61.2
- net GNDPWR: now also J88.1 (Pin_1)
- net GPIO0: now also J6.1 (Pin_1)
- net GPIO1: now also J6.2 (Pin_2)
- net GPIO2: now also J6.3 (Pin_3)
- net GPIO3: now also J6.4 (Pin_4)
- net HOME/HALL_C/GPIO2 renamed HOME/HALL_C
- net Phases/C_VOLTAGE_SENSE: no longer names the net of U1.13 (OA3IN+/AN14/ISRC1/RP50/RC2)
- net QEI_A/HALL_A/GPIO0 renamed QEI_A/HALL_A
- net QEI_B/HALL_B/GPIO1 renamed QEI_B/HALL_B
- net SPI_CLK renamed I2C_SCL
- net I2C_SCL: now also J4.2 (Pin_2); no longer J4.1 (Pin_1)
- net SPI_MISO renamed I2C_SDA
- net I2C_SDA: now also J4.3 (Pin_3); no longer J4.2 (Pin_2)
- net SPI_MOSI: no longer names the net of U1.25 (PGC3/RP38/RB6)
- net SPI_MOSI: no longer J4.3 (Pin_3)
- net SPI_SS: no longer names the net of U1.26 (TDO/AN2/RP39/RB7)
- net SPI_SS: no longer J4.4 (Pin_4)
- no-connect marks 3 -> 8
Other:
- sheet Phases ports: added none; removed C_VOLTAGE_SENSE
- note added: "Control board power + I2C"
- note added: "GPIO / I2C address select"
- note removed: "Control board power"
- note removed: "GPIO"
- note removed: "SPI comms"
- moved on the sheet: J4
