File: esc/singlebridge.kicad_sch (KiCad schematic)
At the start: 10 parts

Commit message: Finished layout
Parts:
- removed Q? (x2): Q_NMOS_DGS, symbol Device:Q_NMOS_DGS
- added Q23, Q24: Q_NMOS_GDS, Package_TO_SOT_SMD:TO-252-2, symbol Device:Q_NMOS_GDS
- C45: renamed from C?; footprint (none) -> Capacitor_SMD:C_0603_1608Metric
- C46: renamed from C?; footprint (none) -> Capacitor_SMD:C_0805_2012Metric
- D36, D37, D38: renamed from D?; value D -> 1N5819WS; footprint (none) -> Diode_SMD:D_SOD-323
- R55, R56: renamed from R?; value R -> 15; footprint (none) -> Resistor_SMD:R_0603_1608Metric
- U18: renamed from U?; footprint (none) -> Package_SO:SOP-8_3.9x4.9mm_P1.27mm
Connections:
- net BRIDGE_HIGH: now also Q23.2 (D)
- net BRIDGE_LOW: now also Q24.3 (S)
- net BRIDGE_OUT: now also Q23.3 (S), Q24.2 (D)
- net at D38.2 (A), R56.2: now also Q24.1 (G)
- net at D37.2 (A), R55.2: now also Q23.1 (G)
Changed lines of the file:
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@@
   (symbol (lib_id "power:+12V") (at 116.205 71.755 0)
     (in_bom yes) (on_board yes) (fields_autoplaced)
-    (property "Reference" "#PWR?" (id 0) (at 116.205 75.565 0)
+    (property "Reference" "#PWR0182" (id 0) (at 116.205 75.565 0)
       (effects (font (size 1.27 1.27)) hide)
     )
@@
   (symbol (lib_id "Device:C") (at 104.14 97.79 0)
     (in_bom yes) (on_board yes)
-    (property "Reference" "C?" (id 0) (at 96.52 96.52 0)
+    (property "Reference" "C45" (id 0) (at 96.52 96.52 0)
       (effects (font (size 1.27 1.27)) (justify left))
     )
@@
       (effects (font (size 1.27 1.27)) (justify left))
     )
-    (property "Footprint" "" (id 2) (at 105.1052 101.6 0)
+    (property "Footprint" "Capacitor_SMD:C_0603_1608Metric" (id 2) (at 105.1052 101.6 0)
       (effects (font (size 1.27 1.27)) hide)
     )
@@
     (pin "2")
   )
+  (symbol (lib_id "Device:Q_NMOS_GDS") (at 159.385 73.025 0)
+    (in_bom yes) (on_board yes) (fields_autoplaced)
+    (property "Reference" "Q23" (id 0) (at 165.735 71.7549 0)
+      (effects (font (size 1.27 1.27)) (justify left))
+    )
+    (property "Value" "Q_NMOS_GDS" (id 1) (at 165.735 74.2949 0)
+      (effects (font (size 1.27 1.27)) (justify left))
+    )
+    (property "Footprint" "Package_TO_SOT_SMD:TO-252-2" (id 2) (at 164.465 70.485 0)
+      (effects (font (size 1.27 1.27)) hide)
+    )
+    (property "Datasheet" "~" (id 3) (at 159.385 73.025 0)
+      (effects (font (size 1.27 1.27)) hide)
+    )
+    (pin "1")
+    (pin "2")
+    (pin "3")
+  )
   (symbol (lib_id "Driver_FET:IR2103") (at 116.205 89.535 0)
     (in_bom yes) (on_board yes)
-    (property "Reference" "U?" (id 0) (at 122.555 101.6 0)
+    (property "Reference" "U18" (id 0) (at 122.555 101.6 0)
       (effects (font (size 1.27 1.27)) (justify left))
     )
@@
       (effects (font (size 1.27 1.27)) (justify left))
     )
-    (property "Footprint" "" (id 2) (at 116.205 89.535 0)
+    (property "Footprint" "Package_SO:SOP-8_3.9x4.9mm_P1.27mm" (id 2) (at 116.205 89.535 0)
       (effects (font (size 1.27 1.27) italic) hide)
     )
@@
   (symbol (lib_id "Device:C") (at 126.365 89.535 0)
     (in_bom yes) (on_board yes) (fields_autoplaced)
-    (property "Reference" "C?" (id 0) (at 129.54 88.2649 0)
+    (property "Reference" "C46" (id 0) (at 129.54 88.2649 0)
       (effects (font (size 1.27 1.27)) (justify left))
     )
@@
       (effects (font (size 1.27 1.27)) (justify left))
     )
-    (property "Footprint" "" (id 2) (at 127.3302 93.345 0)
+    (property "Footprint" "Capacitor_SMD:C_0805_2012Metric" (id 2) (at 127.3302 93.345 0)
       (effects (font (size 1.27 1.27)) hide)
     )
@@
     (pin "2")
   )
-  (symbol (lib_id "Device:Q_NMOS_DGS") (at 159.385 104.775 0)
-    (in_bom yes) (on_board yes) (fields_autoplaced)
-    (property "Reference" "Q?" (id 0) (at 165.735 103.5049 0)
-      (effects (font (size 1.27 1.27)) (justify left))
-    )
-    (property "Value" "Q_NMOS_DGS" (id 1) (at 165.735 106.0449 0)
-      (effects (font (size 1.27 1.27)) (justify left))
-    )
-    (property "Footprint" "" (id 2) (at 164.465 102.235 0)
-      (effects (font (size 1.27 1.27)) hide)
-    )
-    (property "Datasheet" "~" (id 3) (at 159.385 104.775 0)
-      (effects (font (size 1.27 1.27)) hide)
-    )
-    (pin "1")
-    (pin "2")
-    (pin "3")
-  )
-  (symbol (lib_id "Device:Q_NMOS_DGS") (at 159.385 73.025 0)
-    (in_bom yes) (on_board yes) (fields_autoplaced)
-    (property "Reference" "Q?" (id 0) (at 165.735 71.7549 0)
-      (effects (font (size 1.27 1.27)) (justify left))
-    )
-    (property "Value" "Q_NMOS_DGS" (id 1) (at 165.735 74.2949 0)
-      (effects (font (size 1.27 1.27)) (justify left))
-    )
-    (property "Footprint" "" (id 2) (at 164.465 70.485 0)
-      (effects (font (size 1.27 1.27)) hide)
-    )
-    (property "Datasheet" "~" (id 3) (at 159.385 73.025 0)
-      (effects (font (size 1.27 1.27)) hide)
-    )
-    (pin "1")
-    (pin "2")
-    (pin "3")
-  )
   (symbol (lib_id "Device:D") (at 142.875 77.47 0)
     (in_bom yes) (on_board yes)
-    (property "Reference" "D?" (id 0) (at 142.875 82.55 0))
-    (property "Value" "D" (id 1) (at 142.875 80.645 0))
-    (property "Footprint" "" (id 2) (at 142.875 77.47 0)
+    (property "Reference" "D37" (id 0) (at 142.875 82.55 0))
+    (property "Value" "1N5819WS" (id 1) (at 142.875 80.645 0))
+    (property "Footprint" "Diode_SMD:D_SOD-323" (id 2) (at 142.875 77.47 0)
       (effects (font (size 1.27 1.27)) hide)
     )
@@
   (symbol (lib_id "power:GNDPWR") (at 116.205 104.775 0)
     (in_bom yes) (on_board yes) (fields_autoplaced)
-    (property "Reference" "#PWR?" (id 0) (at 116.205 109.855 0)
+    (property "Reference" "#PWR0181" (id 0) (at 116.205 109.855 0)
       (effects (font (size 1.27 1.27)) hide)
     )
@@
     (pin "1")
   )
+  (symbol (lib_id "Device:Q_NMOS_GDS") (at 159.385 104.775 0)
+    (in_bom yes) (on_board yes) (fields_autoplaced)
+    (property "Reference" "Q24" (id 0) (at 165.735 103.5049 0)
+      (effects (font (size 1.27 1.27)) (justify left))
+    )
+    (property "Value" "Q_NMOS_GDS" (id 1) (at 165.735 106.0449 0)
+      (effects (font (size 1.27 1.27)) (justify left))
+    )
+    (property "Footprint" "Package_TO_SOT_SMD:TO-252-2" (id 2) (at 164.465 102.235 0)
+      (effects (font (size 1.27 1.27)) hide)
+    )
+    (property "Datasheet" "~" (id 3) (at 159.385 104.775 0)
+      (effects (font (size 1.27 1.27)) hide)
+    )
+    (pin "1")
+    (pin "2")
+    (pin "3")
+  )
   (symbol (lib_id "Device:D") (at 142.875 100.33 0)
     (in_bom yes) (on_board yes)
-    (property "Reference" "D?" (id 0) (at 144.78 97.79 0))
-    (property "Value" "D" (id 1) (at 141.605 97.79 0))
-    (property "Footprint" "" (id 2) (at 142.875 100.33 0)
+    (property "Reference" "D38" (id 0) (at 144.78 97.79 0))
+    (property "Value" "1N5819WS" (id 1) (at 141.605 97.79 0))
+    (property "Footprint" "Diode_SMD:D_SOD-323" (id 2) (at 142.875 100.33 0)
       (effects (font (size 1.27 1.27)) hide)
     )
@@
   (symbol (lib_id "Device:D") (at 121.92 74.295 180)
     (in_bom yes) (on_board yes) (fields_autoplaced)
-    (property "Reference" "D?" (id 0) (at 121.92 67.945 0))
-    (property "Value" "D" (id 1) (at 121.92 70.485 0))
-    (property "Footprint" "" (id 2) (at 121.92 74.295 0)
+    (property "Reference" "D36" (id 0) (at 121.92 67.31 0))
+    (property "Value" "1N5819WS" (id 1) (at 121.92 69.85 0))
+    (property "Footprint" "Diode_SMD:D_SOD-323" (id 2) (at 121.92 74.295 0)
       (effects (font (size 1.27 1.27)) hide)
     )
@@
   (symbol (lib_id "Device:R") (at 142.875 104.775 90)
     (in_bom yes) (on_board yes)
-    (property "Reference" "R?" (id 0) (at 142.875 106.68 90))
-    (property "Value" "R" (id 1) (at 142.24 108.585 90))
-    (property "Footprint" "" (id 2) (at 142.875 106.553 90)
+    (property "Reference" "R56" (id 0) (at 142.875 106.68 90))
+    (property "Value" "15" (id 1) (at 142.24 108.585 90))
+    (property "Footprint" "Resistor_SMD:R_0603_1608Metric" (id 2) (at 142.875 106.553 90)
       (effects (font (size 1.27 1.27)) hide)
     )
@@
   (symbol (lib_id "Device:R") (at 142.875 73.025 90)
     (in_bom yes) (on_board yes)
-    (property "Reference" "R?" (id 0) (at 142.875 69.215 90))
-    (property "Value" "R" (id 1) (at 142.875 71.12 90))
-    (property "Footprint" "" (id 2) (at 142.875 74.803 90)
+    (property "Reference" "R55" (id 0) (at 142.875 69.215 90))
+    (property "Value" "15" (id 1) (at 142.875 71.12 90))
+    (property "Footprint" "Resistor_SMD:R_0603_1608Metric" (id 2) (at 142.875 74.803 90)
       (effects (font (size 1.27 1.27)) hide)
     )

Commit message: Finished design - first submission
Parts:
- renumbered C45 to C23, C46 to C24, D36 to D3, D37 to D4, D38 to D5, Q23 to Q1, Q24 to Q2, R55 to R33, R56 to R34, U18 to U7
Changed lines of the file:
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@@
     (effects (font (size 1.27 1.27)) (justify left))
   )
-  (symbol (lib_id "power:+12V") (at 116.205 71.755 0)
+  (symbol (lib_id "power:+12V") (at 116.205 71.755 0) (unit 1)
     (in_bom yes) (on_board yes) (fields_autoplaced)
-    (property "Reference" "#PWR0182" (id 0) (at 116.205 75.565 0)
+    (property "Reference" "#PWR0160" (id 0) (at 116.205 75.565 0)
       (effects (font (size 1.27 1.27)) hide)
     )
@@
     (pin "1")
   )
-  (symbol (lib_id "Device:C") (at 104.14 97.79 0)
+  (symbol (lib_id "Device:C") (at 104.14 97.79 0) (unit 1)
     (in_bom yes) (on_board yes)
-    (property "Reference" "C45" (id 0) (at 96.52 96.52 0)
+    (property "Reference" "C23" (id 0) (at 96.52 96.52 0)
       (effects (font (size 1.27 1.27)) (justify left))
     )
@@
     (pin "2")
   )
-  (symbol (lib_id "Device:Q_NMOS_GDS") (at 159.385 73.025 0)
+  (symbol (lib_id "Device:Q_NMOS_GDS") (at 159.385 73.025 0) (unit 1)
     (in_bom yes) (on_board yes) (fields_autoplaced)
-    (property "Reference" "Q23" (id 0) (at 165.735 71.7549 0)
+    (property "Reference" "Q1" (id 0) (at 165.735 71.7549 0)
       (effects (font (size 1.27 1.27)) (justify left))
     )
@@
     (pin "3")
   )
-  (symbol (lib_id "Driver_FET:IR2103") (at 116.205 89.535 0)
+  (symbol (lib_id "Driver_FET:IR2103") (at 116.205 89.535 0) (unit 1)
     (in_bom yes) (on_board yes)
-    (property "Reference" "U18" (id 0) (at 122.555 101.6 0)
+    (property "Reference" "U7" (id 0) (at 122.555 101.6 0)
       (effects (font (size 1.27 1.27)) (justify left))
     )
@@
     (pin "8")
   )
-  (symbol (lib_id "Device:C") (at 126.365 89.535 0)
+  (symbol (lib_id "Device:C") (at 126.365 89.535 0) (unit 1)
     (in_bom yes) (on_board yes) (fields_autoplaced)
-    (property "Reference" "C46" (id 0) (at 129.54 88.2649 0)
+    (property "Reference" "C24" (id 0) (at 129.54 88.2649 0)
       (effects (font (size 1.27 1.27)) (justify left))
     )
@@
     (pin "2")
   )
-  (symbol (lib_id "Device:D") (at 142.875 77.47 0)
+  (symbol (lib_id "Device:D") (at 142.875 77.47 0) (unit 1)
     (in_bom yes) (on_board yes)
-    (property "Reference" "D37" (id 0) (at 142.875 82.55 0))
+    (property "Reference" "D4" (id 0) (at 142.875 82.55 0))
     (property "Value" "1N5819WS" (id 1) (at 142.875 80.645 0))
     (property "Footprint" "Diode_SMD:D_SOD-323" (id 2) (at 142.875 77.47 0)
@@
     (pin "2")
   )
-  (symbol (lib_id "power:GNDPWR") (at 116.205 104.775 0)
+  (symbol (lib_id "power:GNDPWR") (at 116.205 104.775 0) (unit 1)
     (in_bom yes) (on_board yes) (fields_autoplaced)
-    (property "Reference" "#PWR0181" (id 0) (at 116.205 109.855 0)
+    (property "Reference" "#PWR0159" (id 0) (at 116.205 109.855 0)
       (effects (font (size 1.27 1.27)) hide)
     )
@@
     (pin "1")
   )
-  (symbol (lib_id "Device:Q_NMOS_GDS") (at 159.385 104.775 0)
+  (symbol (lib_id "Device:Q_NMOS_GDS") (at 159.385 104.775 0) (unit 1)
     (in_bom yes) (on_board yes) (fields_autoplaced)
-    (property "Reference" "Q24" (id 0) (at 165.735 103.5049 0)
+    (property "Reference" "Q2" (id 0) (at 165.735 103.5049 0)
       (effects (font (size 1.27 1.27)) (justify left))
     )
@@
     (pin "3")
   )
-  (symbol (lib_id "Device:D") (at 142.875 100.33 0)
+  (symbol (lib_id "Device:D") (at 142.875 100.33 0) (unit 1)
     (in_bom yes) (on_board yes)
-    (property "Reference" "D38" (id 0) (at 144.78 97.79 0))
+    (property "Reference" "D5" (id 0) (at 144.78 97.79 0))
     (property "Value" "1N5819WS" (id 1) (at 141.605 97.79 0))
     (property "Footprint" "Diode_SMD:D_SOD-323" (id 2) (at 142.875 100.33 0)
@@
     (pin "2")
   )
-  (symbol (lib_id "Device:D") (at 121.92 74.295 180)
+  (symbol (lib_id "Device:D") (at 121.92 74.295 180) (unit 1)
     (in_bom yes) (on_board yes) (fields_autoplaced)
-    (property "Reference" "D36" (id 0) (at 121.92 67.31 0))
+    (property "Reference" "D3" (id 0) (at 121.92 67.31 0))
     (property "Value" "1N5819WS" (id 1) (at 121.92 69.85 0))
     (property "Footprint" "Diode_SMD:D_SOD-323" (id 2) (at 121.92 74.295 0)
@@
     (pin "2")
   )
-  (symbol (lib_id "Device:R") (at 142.875 104.775 90)
+  (symbol (lib_id "Device:R") (at 142.875 104.775 90) (unit 1)
     (in_bom yes) (on_board yes)
-    (property "Reference" "R56" (id 0) (at 142.875 106.68 90))
+    (property "Reference" "R34" (id 0) (at 142.875 106.68 90))
     (property "Value" "15" (id 1) (at 142.24 108.585 90))
     (property "Footprint" "Resistor_SMD:R_0603_1608Metric" (id 2) (at 142.875 106.553 90)
@@
     (pin "2")
   )
-  (symbol (lib_id "Device:R") (at 142.875 73.025 90)
+  (symbol (lib_id "Device:R") (at 142.875 73.025 90) (unit 1)
     (in_bom yes) (on_board yes)
-    (property "Reference" "R55" (id 0) (at 142.875 69.215 90))
+    (property "Reference" "R33" (id 0) (at 142.875 69.215 90))
     (property "Value" "15" (id 1) (at 142.875 71.12 90))
     (property "Footprint" "Resistor_SMD:R_0603_1608Metric" (id 2) (at 142.875 74.803 90)

Commit message: Some stuff
Parts:
- added J12, J13, J14: Conn_01x01, Library:SmallPin, symbol Connector_Generic:Conn_01x01
- added J15, J16, J17: Conn_01x01, Library:SmallPad, symbol Connector_Generic:Conn_01x01
- D3, D4, D5: footprint Diode_SMD:D_SOD-323 -> Diode_SMD:D_SOD-323_HandSoldering
Connections:
- net BRIDGE_OUT: now also J16.1 (Pin_1); no longer C24.2, U7.6 (VS)
- net at D4.2 (A), R33.2: now also J12.1 (Pin_1); no longer Q1.1 (G)
- net at D5.2 (A), R34.2: now also J14.1 (Pin_1); no longer Q2.1 (G)
- new net: C24.2, J13.1 (Pin_1), U7.6 (VS)
- new net: J15.1 (Pin_1), Q1.1 (G)
- new net: J17.1 (Pin_1), Q2.1 (G)
Other:
- note added: "Control board"
- note added: "Power board"
- moved on the sheet: C23, C24, D3, D4, D5, Q1, Q2, R33, R34, U7

Commit message: Pretty much finished new design
Connections:
- net GNDPWR renamed GND
Changed lines of the file:
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@@
+    (pin "1")
+  )
+  (symbol (lib_id "power:GND") (at 100.965 104.775 0) (unit 1)
+    (in_bom yes) (on_board yes) (fields_autoplaced)
+    (property "Reference" "#PWR?" (id 0) (at 100.965 111.125 0)
+      (effects (font (size 1.27 1.27)) hide)
+    )
+    (property "Value" "GND" (id 1) (at 100.965 109.22 0))
+    (property "Footprint" "" (id 2) (at 100.965 104.775 0)
+      (effects (font (size 1.27 1.27)) hide)
+    )
+    (property "Datasheet" "" (id 3) (at 100.965 104.775 0)
+      (effects (font (size 1.27 1.27)) hide)
+    )
     (pin "1")
   )
@@
     (pin "2")
   )
-  (symbol (lib_id "power:GNDPWR") (at 100.965 104.775 0) (unit 1)
-    (in_bom yes) (on_board yes) (fields_autoplaced)
-    (property "Reference" "#PWR0159" (id 0) (at 100.965 109.855 0)
-      (effects (font (size 1.27 1.27)) hide)
-    )
-    (property "Value" "GNDPWR" (id 1) (at 100.838 109.22 0))
-    (property "Footprint" "" (id 2) (at 100.965 106.045 0)
-      (effects (font (size 1.27 1.27)) hide)
-    )
-    (property "Datasheet" "" (id 3) (at 100.965 106.045 0)
-      (effects (font (size 1.27 1.27)) hide)
-    )
-    (pin "1")
-  )
   (symbol (lib_id "Device:Q_NMOS_GDS") (at 176.53 104.775 0) (unit 1)
