File: esc/esc.kicad_pcb (KiCad board)
At the start: 4 copper layers, 99.6 x 48.3 mm, 196 parts, among them J3 Conn_01x05, J4 Conn_01x05, J5 Conn_01x04, Q1 Q_NMOS_GDS, Q10 Q_NMOS_GDS, Q11 Q_NMOS_GDS, Q12 Q_NMOS_GDS, Q13 Q_NMOS_GDS, Q14 Q_NMOS_GDS, Q15 Q_NMOS_GDS, Q16 Q_NMOS_GDS, Q17 Q_NMOS_GDS, Q18 Q_NMOS_GDS, Q19 Q_NMOS_GDS, Q2 Q_NMOS_GDS, Q20 Q_NMOS_GDS, Q21 Q_NMOS_GDS, Q22 Q_NMOS_GDS, Q23 Q_NMOS_GDS, Q24 Q_NMOS_GDS, Q3 Q_NMOS_GDS, Q4 Q_NMOS_GDS, Q5 Q_NMOS_GDS, Q6 Q_NMOS_GDS, Q7 Q_NMOS_GDS, Q8 Q_NMOS_GDS, Q9 Q_NMOS_GDS, SW1 SW_SPDT, SW2 SW_SPDT, SW3 SW_SPDT, U1 dsPIC33CK64MC103, U10 EG2131, U11 EG2131, U12 EG2131, U13 EG2131, U14 EG2131, U15 EG2131, U16 EG2131, U17 EG2131, U18 EG2131, U2 GS8051, U3 GS8051, U4 MC34063AD, U5 MC34063AD, U6 AP1117-ADJ, U7 EG2131, U8 EG2131, U9 EG2131

Commit message: Finished design - first submission
Parts:
- added TP10: TestPoint, TestPoint:TestPoint_Pad_1.0x1.0mm, F.Cu at (175.5, 50.8)
- added TP11: TestPoint, TestPoint:TestPoint_Pad_1.0x1.0mm, F.Cu at (169.9, 56.9)
- added TP12: TestPoint, TestPoint:TestPoint_Pad_1.0x1.0mm, F.Cu at (177.5, 65.8)
- added TP13: TestPoint, TestPoint:TestPoint_Pad_1.0x1.0mm, B.Cu at (172.7, 74.4)
- added TP14: TestPoint, TestPoint:TestPoint_Pad_1.0x1.0mm, B.Cu at (172.7, 76.7)
- added TP16: TestPoint, TestPoint:TestPoint_Pad_1.0x1.0mm, B.Cu at (177.8, 64.0)
- added TP17: TestPoint, TestPoint:TestPoint_Pad_1.0x1.0mm, B.Cu at (190.5, 38.9)
- added TP18: TestPoint, TestPoint:TestPoint_Pad_1.0x1.0mm, B.Cu at (175.0, 65.8)
- added TP19: TestPoint, TestPoint:TestPoint_Pad_1.0x1.0mm, B.Cu at (173.7, 60.2)
- added TP20: TestPoint, TestPoint:TestPoint_Pad_1.0x1.0mm, B.Cu at (170.2, 66.5)
- added TP21: TestPoint, TestPoint:TestPoint_Pad_1.0x1.0mm, B.Cu at (189.2, 36.3)
- added TP3: TestPoint, TestPoint:TestPoint_Pad_1.0x1.0mm, B.Cu at (197.9, 55.6)
- added TP4: TestPoint, TestPoint:TestPoint_Pad_1.0x1.0mm, B.Cu at (176.8, 69.3)
- added TP5: TestPoint, TestPoint:TestPoint_Pad_1.0x1.0mm, B.Cu at (176.8, 71.6)
- added TP6: TestPoint, TestPoint:TestPoint_Pad_1.0x1.0mm, B.Cu at (170.2, 61.7)
- added TP7: TestPoint, TestPoint:TestPoint_Pad_1.0x1.0mm, B.Cu at (170.2, 64.0)
- added TP8: TestPoint, TestPoint:TestPoint_Pad_1.0x1.0mm, B.Cu at (181.4, 69.3)
- added TP9: TestPoint, TestPoint:TestPoint_Pad_1.0x1.0mm, B.Cu at (181.4, 71.6)
Routing:
- net /Phases/C_HIN: track 78.9 -> 86.6 mm
- net /Phases/~{C_LIN}: track 76.6 -> 83.6 mm
- net +12V: track 110.1 -> 114.1 mm
- net /LV_SUPPLY: track 0.00 -> 3.65 mm
- net /Phases/~{A_LIN}: track 61.9 -> 64.8 mm
- net /Phases/A_HIN: track 61.0 -> 63.8 mm
- net /Phases/B_VOLTAGE_SENSE: track 28.3 -> 31.0 mm
- net +3.3VA: track 67.9 -> 70.5 mm
- net +5V: track 36.0 -> 37.8 mm
- net /Phases/A_VOLTAGE_SENSE: track 33.0 -> 34.8 mm
- net +3V3: track 84.8 -> 86.5 mm
- net /Phases/~{B_LIN}: track 46.9 -> 48.1 mm
- net GND: track 37.3 -> 38.3 mm, vias 3 -> 4
- net GNDA: track 79.4 -> 80.1 mm
- net /Phases/B_HIN: track 49.7 -> 50.3 mm

Commit message: Working version
Changed lines of the file:
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@@
       (outputformat 1)
       (mirror false)
-      (drillshape 1)
+      (drillshape 0)
       (scaleselection 1)
-      (outputdirectory "")
+      (outputdirectory "out")
     )
   )
@@
     (fp_line (start -2.5 2.5) (end -2.5 -1.5) (layer "F.Fab") (width 0.1))
     (pad "" connect roundrect (at -2.5 -2.5) (size 0.85 0.85) (layers "F.Cu" "F.Mask") (roundrect_rratio 0.15))
-    (pad "" smd roundrect (at -1.27 0) (size 1.02 1.02) (layers "F.Paste") (roundrect_rratio 0.245098))
-    (pad "" smd roundrect (at 1.27 1.27) (size 1.02 1.02) (layers "F.Paste") (roundrect_rratio 0.245098))
-    (pad "" smd roundrect (at 1.27 0) (size 1.02 1.02) (layers "F.Paste") (roundrect_rratio 0.245098))
-    (pad "" smd roundrect (at 0 1.27) (size 1.02 1.02) (layers "F.Paste") (roundrect_rratio 0.245098))
-    (pad "" smd roundrect (at 0 0) (size 1.02 1.02) (layers "F.Paste") (roundrect_rratio 0.245098))
-    (pad "" smd roundrect (at -1.27 -1.27) (size 1.02 1.02) (layers "F.Paste") (roundrect_rratio 0.245098))
+    (pad "" smd roundrect (at -1.27 0) (size 1.02 1.02) (layers "F.Paste") (roundrect_rratio 0.2450980392))
+    (pad "" smd roundrect (at 1.27 1.27) (size 1.02 1.02) (layers "F.Paste") (roundrect_rratio 0.2450980392))
+    (pad "" smd roundrect (at 1.27 0) (size 1.02 1.02) (layers "F.Paste") (roundrect_rratio 0.2450980392))
+    (pad "" smd roundrect (at 0 1.27) (size 1.02 1.02) (layers "F.Paste") (roundrect_rratio 0.2450980392))
+    (pad "" smd roundrect (at 0 0) (size 1.02 1.02) (layers "F.Paste") (roundrect_rratio 0.2450980392))
+    (pad "" smd roundrect (at -1.27 -1.27) (size 1.02 1.02) (layers "F.Paste") (roundrect_rratio 0.2450980392))
     (pad "" connect roundrect (at 2.5 -2.5) (size 0.85 0.85) (layers "F.Cu" "F.Mask") (roundrect_rratio 0.15))
-    (pad "" smd roundrect (at -1.27 1.27) (size 1.02 1.02) (layers "F.Paste") (roundrect_rratio 0.245098))
+    (pad "" smd roundrect (at -1.27 1.27) (size 1.02 1.02) (layers "F.Paste") (roundrect_rratio 0.2450980392))
     (pad "" connect roundrect (at 2.5 2.5) (size 0.85 0.85) (layers "F.Cu" "F.Mask") (roundrect_rratio 0.15))
-    (pad "" smd roundrect (at 0 -1.27) (size 1.02 1.02) (layers "F.Paste") (roundrect_rratio 0.245098))
+    (pad "" smd roundrect (at 0 -1.27) (size 1.02 1.02) (layers "F.Paste") (roundrect_rratio 0.2450980392))
     (pad "" connect roundrect (at -2.5 2.5) (size 0.85 0.85) (layers "F.Cu" "F.Mask") (roundrect_rratio 0.15))
-    (pad "" smd roundrect (at 1.27 -1.27) (size 1.02 1.02) (layers "F.Paste") (roundrect_rratio 0.245098))
+    (pad "" smd roundrect (at 1.27 -1.27) (size 1.02 1.02) (layers "F.Paste") (roundrect_rratio 0.2450980392))
     (pad "1" smd roundrect (at -2.5 -1.6) (size 0.75 0.2) (layers "F.Cu" "F.Paste" "F.Mask") (roundrect_rratio 0.25)
       (net 100 "/Phases/A_HIN") (pinfunction "RP46/PWM1H/RB14") (pintype "bidirectional"))
@@
     (fp_line (start -3.15 -1.6) (end -3.15 1.6) (layer "B.Fab") (width 0.1))
     (fp_line (start 3.15 -1.6) (end -3.15 -1.6) (layer "B.Fab") (width 0.1))
-    (pad "1" smd roundrect (at -2.9625 0 270) (size 1.225 3.35) (layers "B.Cu" "B.Paste" "B.Mask") (roundrect_rratio 0.204082)
+    (pad "1" smd roundrect (at -2.9625 0 270) (size 1.225 3.35) (layers "B.Cu" "B.Paste" "B.Mask") (roundrect_rratio 0.2040816327)
       (net 15 "/Phases/Phase B/BRIDGE_LOW") (pintype "passive"))
-    (pad "2" smd roundrect (at 2.9625 0 270) (size 1.225 3.35) (layers "B.Cu" "B.Paste" "B.Mask") (roundrect_rratio 0.204082)
+    (pad "2" smd roundrect (at 2.9625 0 270) (size 1.225 3.35) (layers "B.Cu" "B.Paste" "B.Mask") (roundrect_rratio 0.2040816327)
       (net 25 "GNDPWR") (pintype "passive"))
     (model "${KICAD6_3DMODEL_DIR}/Resistor_SMD.3dshapes/R_2512_6332Metric.wrl"
@@
     (fp_line (start 3.15 -1.6) (end -3.15 -1.6) (layer "B.Fab") (width 0.1))
     (fp_line (start -3.15 1.6) (end 3.15 1.6) (layer "B.Fab") (width 0.1))
-    (pad "1" smd roundrect (at -2.9625 0 270) (size 1.225 3.35) (layers "B.Cu" "B.Paste" "B.Mask") (roundrect_rratio 0.204082)
+    (pad "1" smd roundrect (at -2.9625 0 270) (size 1.225 3.35) (layers "B.Cu" "B.Paste" "B.Mask") (roundrect_rratio 0.2040816327)
       (net 5 "/Phases/Phase A/BRIDGE_LOW") (pintype "passive"))
-    (pad "2" smd roundrect (at 2.9625 0 270) (size 1.225 3.35) (layers "B.Cu" "B.Paste" "B.Mask") (roundrect_rratio 0.204082)
+    (pad "2" smd roundrect (at 2.9625 0 270) (size 1.225 3.35) (layers "B.Cu" "B.Paste" "B.Mask") (roundrect_rratio 0.2040816327)
       (net 25 "GNDPWR") (pintype "passive"))
     (model "${KICAD6_3DMODEL_DIR}/Resistor_SMD.3dshapes/R_2512_6332Metric.wrl"
@@
     (fp_line (start 3.15 1.6) (end 3.15 -1.6) (layer "B.Fab") (width 0.1))
     (fp_line (start -3.15 1.6) (end 3.15 1.6) (layer "B.Fab") (width 0.1))
-    (pad "1" smd roundrect (at -2.9625 0 270) (size 1.225 3.35) (layers "B.Cu" "B.Paste" "B.Mask") (roundrect_rratio 0.204082)
+    (pad "1" smd roundrect (at -2.9625 0 270) (size 1.225 3.35) (layers "B.Cu" "B.Paste" "B.Mask") (roundrect_rratio 0.2040816327)
       (net 5 "/Phases/Phase A/BRIDGE_LOW") (pintype "passive"))
-    (pad "2" smd roundrect (at 2.9625 0 270) (size 1.225 3.35) (layers "B.Cu" "B.Paste" "B.Mask") (roundrect_rratio 0.204082)
+    (pad "2" smd roundrect (at 2.9625 0 270) (size 1.225 3.35) (layers "B.Cu" "B.Paste" "B.Mask") (roundrect_rratio 0.2040816327)
       (net 25 "GNDPWR") (pintype "passive"))
     (model "${KICAD6_3DMODEL_DIR}/Resistor_SMD.3dshapes/R_2512_6332Metric.wrl"
@@
     (fp_line (start 1.6 -0.8) (end -1.6 -0.8) (layer "B.Fab") (width 0.1))
     (fp_line (start -1.6 -0.8) (end -1.6 0.8) (layer "B.Fab") (width 0.1))
-    (pad "1" smd roundrect (at -1.4625 0 270) (size 1.125 1.75) (layers "B.Cu" "B.Paste" "B.Mask") (roundrect_rratio 0.222222)
+    (pad "1" smd roundrect (at -1.4625 0 270) (size 1.125 1.75) (layers "B.Cu" "B.Paste" "B.Mask") (roundrect_rratio 0.2222222222)
       (net 44 "/Supplies/VIN") (pintype "passive"))
-    (pad "2" smd roundrect (at 1.4625 0 270) (size 1.125 1.75) (layers "B.Cu" "B.Paste" "B.Mask") (roundrect_rratio 0.222222)
+    (pad "2" smd roundrect (at 1.4625 0 270) (size 1.125 1.75) (layers "B.Cu" "B.Paste" "B.Mask") (roundrect_rratio 0.2222222222)
       (net 40 "Net-(R24-Pad2)") (pintype "passive"))
     (model "${KICAD6_3DMODEL_DIR}/Resistor_SMD.3dshapes/R_1206_3216Metric.wrl"
@@
     (fp_line (start 3.15 1.6) (end 3.15 -1.6) (layer "B.Fab") (width 0.1))
     (fp_line (start -3.15 -1.6) (end -3.15 1.6) (layer "B.Fab") (width 0.1))
-    (pad "1" smd roundrect (at -2.9625 0 270) (size 1.225 3.35) (layers "B.Cu" "B.Paste" "B.Mask") (roundrect_rratio 0.204082)
+    (pad "1" smd roundrect (at -2.9625 0 270) (size 1.225 3.35) (layers "B.Cu" "B.Paste" "B.Mask") (roundrect_rratio 0.2040816327)
       (net 15 "/Phases/Phase B/BRIDGE_LOW") (pintype "passive"))
-    (pad "2" smd roundrect (at 2.9625 0 270) (size 1.225 3.35) (layers "B.Cu" "B.Paste" "B.Mask") (roundrect_rratio 0.204082)
+    (pad "2" smd roundrect (at 2.9625 0 270) (size 1.225 3.35) (layers "B.Cu" "B.Paste" "B.Mask") (roundrect_rratio 0.2040816327)
       (net 25 "GNDPWR") (pintype "passive"))
     (model "${KICAD6_3DMODEL_DIR}/Resistor_SMD.3dshapes/R_2512_6332Metric.wrl"
@@
     (fp_line (start 1.6 -0.8) (end -1.6 -0.8) (layer "B.Fab") (width 0.1))
     (fp_line (start 1.6 0.8) (end 1.6 -0.8) (layer "B.Fab") (width 0.1))
-    (pad "1" smd roundrect (at -1.4625 0 270) (size 1.125 1.75) (layers "B.Cu" "B.Paste" "B.Mask") (roundrect_rratio 0.222222)
+    (pad "1" smd roundrect (at -1.4625 0 270) (size 1.125 1.75) (layers "B.Cu" "B.Paste" "B.Mask") (roundrect_rratio 0.2222222222)
       (net 48 "+5V") (pintype "passive"))
-    (pad "2" smd roundrect (at 1.4625 0 270) (size 1.125 1.75) (layers "B.Cu" "B.Paste" "B.Mask") (roundrect_rratio 0.222222)
+    (pad "2" smd roundrect (at 1.4625 0 270) (size 1.125 1.75) (layers "B.Cu" "B.Paste" "B.Mask") (roundrect_rratio 0.2222222222)
       (net 49 "Net-(L2-Pad1)") (pintype "passive"))
     (model "${KICAD6_3DMODEL_DIR}/Resistor_SMD.3dshapes/R_1206_3216Metric.wrl"
@@
     (fp_line (start 3.15 1.6) (end 3.15 -1.6) (layer "B.Fab") (width 0.1))
     (fp_line (start -3.15 1.6) (end 3.15 1.6) (layer "B.Fab") (width 0.1))
-    (pad "1" smd roundrect (at -2.9625 0 270) (size 1.225 3.35) (layers "B.Cu" "B.Paste" "B.Mask") (roundrect_rratio 0.204082)
+    (pad "1" smd roundrect (at -2.9625 0 270) (size 1.225 3.35) (layers "B.Cu" "B.Paste" "B.Mask") (roundrect_rratio 0.2040816327)
       (net 15 "/Phases/Phase B/BRIDGE_LOW") (pintype "passive"))
-    (pad "2" smd roundrect (at 2.9625 0 270) (size 1.225 3.35) (layers "B.Cu" "B.Paste" "B.Mask") (roundrect_rratio 0.204082)
+    (pad "2" smd roundrect (at 2.9625 0 270) (size 1.225 3.35) (layers "B.Cu" "B.Paste" "B.Mask") (roundrect_rratio 0.2040816327)
       (net 25 "GNDPWR") (pintype "passive"))
     (model "${KICAD6_3DMODEL_DIR}/Resistor_SMD.3dshapes/R_2512_6332Metric.wrl"
@@
     (fp_line (start -3.15 -1.6) (end -3.15 1.6) (layer "B.Fab") (width 0.1))
     (fp_line (start 3.15 -1.6) (end -3.15 -1.6) (layer "B.Fab") (width 0.1))
-    (pad "1" smd roundrect (at -2.9625 0 270) (size 1.225 3.35) (layers "B.Cu" "B.Paste" "B.Mask") (roundrect_rratio 0.204082)
+    (pad "1" smd roundrect (at -2.9625 0 270) (size 1.225 3.35) (layers "B.Cu" "B.Paste" "B.Mask") (roundrect_rratio 0.2040816327)
       (net 5 "/Phases/Phase A/BRIDGE_LOW") (pintype "passive"))
-    (pad "2" smd roundrect (at 2.9625 0 270) (size 1.225 3.35) (layers "B.Cu" "B.Paste" "B.Mask") (roundrect_rratio 0.204082)
+    (pad "2" smd roundrect (at 2.9625 0 270) (size 1.225 3.35) (layers "B.Cu" "B.Paste" "B.Mask") (roundrect_rratio 0.2040816327)
       (net 25 "GNDPWR") (pintype "passive"))
     (model "${KICAD6_3DMODEL_DIR}/Resistor_SMD.3dshapes/R_2512_6332Metric.wrl"

Commit message: Some stuff
Parts:
- removed C47: 1u, Capacitor_SMD:C_0603_1608Metric
- removed D1, D2: SS14, Diode_SMD:D_SMA
- removed J4: Conn_01x05, Connector_PinHeader_2.54mm:PinHeader_1x05_P2.54mm_Vertical
- removed J5: Conn_01x04, Connector_PinHeader_2.54mm:PinHeader_1x04_P2.54mm_Vertical
- removed L1, L2, L3: 100u, Inductor_SMD:L_Sumida_CR75
- removed NT2: NetTie_2, footprints:Nettie2
- removed SW1, SW2, SW3: SW_SPDT, Connector_PinHeader_2.54mm:PinHeader_1x03_P2.54mm_Vertical
- removed TP10, TP11, TP12, TP13, TP14, TP16, TP17, TP18, TP19, TP20, TP21, TP3: TestPoint, TestPoint:TestPoint_Pad_1.0x1.0mm
- removed U5: MC34063AD, Package_SO:SOIC-8_3.9x4.9mm_P1.27mm
- removed U6: AP1117-ADJ, Package_TO_SOT_SMD:SOT-223-3_TabPin2
- added J10: Conn_01x01, Library:SmallPin, F.Cu at (107.2, 125.7)
- added J11: Conn_01x01, Library:SmallPin, F.Cu at (132.8, 125.7)
- added J12: Conn_01x01, Library:SmallPin, F.Cu at (108.2, 116.3)
- added J13: Conn_01x01, Library:SmallPin, F.Cu at (108.2, 111.8)
- added J14: Conn_01x01, Library:SmallPin, F.Cu at (97.8, 116.3)
- added J17: Conn_01x01, Library:SmallPad, F.Cu at (53.1, 116.3)
- added J18: Conn_01x01, Library:SmallPin, F.Cu at (108.2, 109.2)
- added J19: Conn_01x01, Library:SmallPin, F.Cu at (108.2, 104.6)
- added J20: Conn_01x01, Library:SmallPin, F.Cu at (97.8, 109.2)
- added J23: Conn_01x01, Library:SmallPad, F.Cu at (53.1, 109.2)
- added J24: Conn_01x01, Library:SmallPin, F.Cu at (108.2, 102.1)
- added J25: Conn_01x01, Library:SmallPin, F.Cu at (108.2, 97.5)
- added J26: Conn_01x01, Library:SmallPin, F.Cu at (97.8, 102.1)
- added J29: Conn_01x01, Library:SmallPad, F.Cu at (53.1, 102.1)
- added J30: Conn_01x01, Library:SmallPin, F.Cu at (108.2, 95.0)
- added J31: Conn_01x01, Library:SmallPin, F.Cu at (108.2, 90.4)
- added J32: Conn_01x01, Library:SmallPin, F.Cu at (97.8, 95.0)
- added J35: Conn_01x01, Library:SmallPad, F.Cu at (53.1, 95.0)
- added J36: Conn_01x01, Library:SmallPin, F.Cu at (121.7, 116.3)
- added J37: Conn_01x01, Library:SmallPin, F.Cu at (121.7, 111.8)
- added J38: Conn_01x01, Library:SmallPin, F.Cu at (111.3, 116.3)
- added J41: Conn_01x01, Library:SmallPad, F.Cu at (66.5, 102.1)
- added J42: Conn_01x01, Library:SmallPin, F.Cu at (121.7, 109.2)
- added J43: Conn_01x01, Library:SmallPin, F.Cu at (121.7, 104.6)
- added J44: Conn_01x01, Library:SmallPin, F.Cu at (111.3, 109.2)
- added J47: Conn_01x01, Library:SmallPad, F.Cu at (66.5, 109.2)
- added J48: Conn_01x01, Library:SmallPin, F.Cu at (121.7, 102.1)
- added J49: Conn_01x01, Library:SmallPin, F.Cu at (121.7, 97.5)
- added J50: Conn_01x01, Library:SmallPin, F.Cu at (111.3, 102.1)
- added J53: Conn_01x01, Library:SmallPad, F.Cu at (66.5, 116.3)
- added J54: Conn_01x01, Library:SmallPin, F.Cu at (121.7, 95.0)
- added J55: Conn_01x01, Library:SmallPin, F.Cu at (121.7, 90.4)
- added J56: Conn_01x01, Library:SmallPin, F.Cu at (111.3, 95.0)
- added J59: Conn_01x01, Library:SmallPad, F.Cu at (66.5, 95.0)
- added J60: Conn_01x01, Library:SmallPin, F.Cu at (135.1, 116.3)
- added J61: Conn_01x01, Library:SmallPin, F.Cu at (135.1, 111.8)
- added J62: Conn_01x01, Library:SmallPin, F.Cu at (124.7, 116.3)
- added J65: Conn_01x01, Library:SmallPad, F.Cu at (80.0, 116.3)
- added J66: Conn_01x01, Library:SmallPin, F.Cu at (135.1, 109.2)
- added J67: Conn_01x01, Library:SmallPin, F.Cu at (135.1, 104.6)
- added J68: Conn_01x01, Library:SmallPin, F.Cu at (124.7, 109.2)
- added J7: Conn_01x05, Connector_PinHeader_2.54mm:PinHeader_1x05_P2.54mm_Horizontal, F.Cu at (112.0, 87.8)
- added J71: Conn_01x01, Library:SmallPad, F.Cu at (80.0, 109.2)
- added J72: Conn_01x01, Library:SmallPin, F.Cu at (135.1, 102.1)
- added J73: Conn_01x01, Library:SmallPin, F.Cu at (135.1, 97.5)
- added J74: Conn_01x01, Library:SmallPin, F.Cu at (124.7, 102.1)
- added J77: Conn_01x01, Library:SmallPad, F.Cu at (80.0, 102.1)
- added J78: Conn_01x01, Library:SmallPin, F.Cu at (135.1, 95.0)
- added J79: Conn_01x01, Library:SmallPin, F.Cu at (135.1, 90.4)
- added J8: Conn_01x01, Library:SmallPad, F.Cu at (62.5, 125.7)
- added J80: Conn_01x01, Library:SmallPin, F.Cu at (124.7, 95.0)
- added J83: Conn_01x01, Library:SmallPad, F.Cu at (80.0, 95.0)
- added J84: Conn_01x01, Library:SmallPin, F.Cu at (132.8, 121.2)
- added J85: Conn_01x01, Library:SmallPad, F.Cu at (88.1, 121.2)
- added J86: Conn_01x01, Library:SmallPin, F.Cu at (107.2, 121.2)
- added J87: Conn_01x01, Library:SmallPad, F.Cu at (62.5, 121.2)
- added J88: Conn_01x01, Library:SmallPad, F.Cu at (62.5, 123.4)
- added J89: Conn_01x01, Library:SmallPad, F.Cu at (88.1, 123.4)
- added J9: Conn_01x01, Library:SmallPad, F.Cu at (88.1, 125.7)
- added J90: Conn_01x01, Library:SmallPin, F.Cu at (107.2, 123.4)
- added J91: Conn_01x01, Library:SmallPin, F.Cu at (132.8, 123.4)
- added R59: 3.3k, Resistor_SMD:R_0603_1608Metric, F.Cu at (85.6, 124.2)
- added TP1: TestPoint, TestPoint:TestPoint_Pad_1.0x1.0mm, F.Cu at (82.6, 47.2)
- added TP2: TestPoint, TestPoint:TestPoint_Pad_1.0x1.0mm, F.Cu at (209.5, 98.0)
- C10, C11, C7: value 300p -> 1n
- C12, C13, C23, C24, C25, C26, C27, C28, C29, C30, C35, C36, C37, C38, R57, R58, U10, U13, U14, U2, U3, U7, U8, U9: moved to F.Cu
- C14: value 470u -> 1n; footprint Capacitor_THT:CP_Radial_D10.0mm_P5.00mm -> Capacitor_SMD:C_0603_1608Metric
- C15: value 470p -> 10u; footprint Capacitor_SMD:C_0603_1608Metric -> Capacitor_SMD:C_0805_2012Metric
- C16: value 220u -> 10u; footprint Capacitor_THT:CP_Radial_D8.0mm_P3.50mm -> Capacitor_SMD:C_0805_2012Metric; moved to B.Cu
- C17: value 470u -> 10u; footprint Capacitor_THT:CP_Radial_D10.0mm_P5.00mm -> Capacitor_SMD:C_0805_2012Metric
- C18: value 470p -> 1u
- C19, C20, C21: value 10u -> 1n; footprint Capacitor_SMD:C_0805_2012Metric -> Capacitor_SMD:C_0603_1608Metric
- C22: value 220u -> 10u; footprint Capacitor_THT:CP_Radial_D8.0mm_P3.50mm -> Capacitor_SMD:C_0805_2012Metric
- C8, C9: value C -> 1n; moved to F.Cu
- D10, D11, D12, D13, D14, D21, D22, D23, D24, D25, D26, D3, D4, D5, D6, D7, D8, D9: footprint Diode_SMD:D_SOD-323 -> Diode_SMD:D_SOD-323_HandSoldering
- D15, D16, D17, D18, D19, D20, D27, D28, D29, D30, D31, D32, D33, D34, D35, D36, D37, D38: footprint Diode_SMD:D_SOD-323 -> Diode_SMD:D_SOD-323_HandSoldering; moved to B.Cu
- NT1: value NetTie_3_Tee -> NetTie_2; footprint footprints:Nettie3 -> footprints:Nettie2
- R10, R11, R8, R9: value 100 -> 120; moved to F.Cu
- R12, R14: value 8.2k -> 330
- R13, R15: value 1k -> 330
- R16, R17, R18, R19: value 4.3k -> 3.3k; moved to F.Cu
- R20: value 8.2k -> 1.5k; moved to B.Cu
- R21, R41, R42, R43, R44, R49, R50, R51, R52, R53, R54, R55, R56: moved to B.Cu
- R22, R23: value 2.2k -> 3.3k; moved to F.Cu
- R24, R27: value 0.51 -> 1k; footprint Resistor_SMD:R_1206_3216Metric -> Resistor_SMD:R_0603_1608Metric
- R25: value 3.6k -> 1k
- R26: value 1.2k -> 1k
- R29: value 180 -> 1k
- R30: value R -> 3.3k; moved to F.Cu
- R31: value 13k -> 3.3k; moved to F.Cu
- R32: value 1.5k -> 3.3k; moved to F.Cu
- U4: value MC34063AD -> AP1117-ADJ; footprint Package_SO:SOIC-8_3.9x4.9mm_P1.27mm -> Package_TO_SOT_SMD:SOT-223-3_TabPin2
- moved R31 150.6 mm to (59.9, 124.2), turned to 180 degrees
- moved R30 134.3 mm to (59.9, 121.2)
- moved R32 130.7 mm to (85.6, 121.2), turned to 180 degrees
- moved R57 103.0 mm to (59.9, 125.7), turned to 180 degrees
- moved R17 102.4 mm to (57.7, 123.4), turned to 90 degrees
- moved R16 100.6 mm to (56.9, 121.2), turned to 0 degrees
- moved C16 98.3 mm to (150.1, 147.6), turned to -90 degrees
- moved C12 97.5 mm to (59.9, 122.7), turned to 0 degrees
- moved C8 95.6 mm to (56.1, 123.4), turned to -90 degrees
- moved C15 95.5 mm to (150.1, 151.4), turned to -90 degrees
- moved R22 95.4 mm to (56.9, 125.7)
- moved C3 95.4 mm to (137.7, 153.4)
- moved U1 95.4 mm to (137.4, 158.2)
- moved R1 95.3 mm to (133.1, 158.0)
- moved C1 95.2 mm to (139.2, 162.6)
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Connections:
- C10 pad 1: /Phases/B_VOLTAGE_SENSE -> /GPIO1
- C10 pad 2: GNDA -> GND
- C11 pad 1: /Phases/C_VOLTAGE_SENSE -> /GPIO2
- C11 pad 2: GNDA -> GND
- C12 pad 1: +3.3VA -> Net-(C12-Pad1)
- C12 pad 2: GNDA -> Net-(C12-Pad2)
- C13 pad 1: +3.3VA -> Net-(C13-Pad1)
- C13 pad 2: GNDA -> Net-(C13-Pad2)
- C14 pad 1: /Supplies/VIN -> /GPIO3
- C15 pad 1: Net-(C15-Pad1) -> +5V
- C16 pad 1: Net-(C16-Pad1) -> +3V3
- C17 pad 1: +5V -> +3.3VA
- C17 pad 2: GND -> GNDA
- C18 pad 1: Net-(C18-Pad1) -> +3.3VA
- C18 pad 2: GND -> GNDA
- C19 pad 1: +5V -> /QEI_A/HALL_A/GPIO0
- C20 pad 1: +3V3 -> /QEI_B/HALL_B/GPIO1
- C21 pad 1: +3.3VA -> /HOME/HALL_C/GPIO2
- C21 pad 2: GNDA -> GND
- C22 pad 1: Net-(C22-Pad1) -> +3V3
- C24 pad 2: /Phases/PHASE_A -> Net-(C24-Pad2)
- C26 pad 2: /Phases/PHASE_A -> Net-(C26-Pad2)
- C28 pad 2: /Phases/PHASE_A -> Net-(C28-Pad2)
- C30 pad 2: /Phases/PHASE_A -> Net-(C30-Pad2)
- C32 pad 2: /Phases/PHASE_B -> Net-(C32-Pad2)
- C34 pad 2: /Phases/PHASE_B -> Net-(C34-Pad2)
- C36 pad 2: /Phases/PHASE_B -> Net-(C36-Pad2)
- C38 pad 2: /Phases/PHASE_B -> Net-(C38-Pad2)
- C40 pad 2: /Phases/PHASE_C -> Net-(C40-Pad2)
- C42 pad 2: /Phases/PHASE_C -> Net-(C42-Pad2)
- C44 pad 2: /Phases/PHASE_C -> Net-(C44-Pad2)
- C46 pad 2: /Phases/PHASE_C -> Net-(C46-Pad2)
- C7 pad 1: /Phases/A_VOLTAGE_SENSE -> /GPIO0
- C7 pad 2: GNDA -> GND
- C8 pad 2: GNDA -> Net-(C8-Pad2)
- C9 pad 2: GNDA -> Net-(C9-Pad2)
- NT1 pad 1: GNDPWR -> +3V3
- NT1 pad 2: GNDA -> +3.3VA
- Q1 pad 1: Net-(D4-Pad2) -> Net-(J15-Pad1)
- Q10 pad 1: Net-(D17-Pad2) -> Net-(J41-Pad1)
- Q11 pad 1: Net-(D19-Pad2) -> Net-(J45-Pad1)
- Q12 pad 1: Net-(D20-Pad2) -> Net-(J47-Pad1)
- Q13 pad 1: Net-(D22-Pad2) -> Net-(J51-Pad1)
- Q14 pad 1: Net-(D23-Pad2) -> Net-(J53-Pad1)
- Q15 pad 1: Net-(D25-Pad2) -> Net-(J57-Pad1)
- Q16 pad 1: Net-(D26-Pad2) -> Net-(J59-Pad1)
- Q17 pad 1: Net-(D28-Pad2) -> Net-(J63-Pad1)
- Q18 pad 1: Net-(D29-Pad2) -> Net-(J65-Pad1)
- Q19 pad 1: Net-(D31-Pad2) -> Net-(J69-Pad1)
- Q2 pad 1: Net-(D5-Pad2) -> Net-(J17-Pad1)
- Q20 pad 1: Net-(D32-Pad2) -> Net-(J71-Pad1)
- Q21 pad 1: Net-(D34-Pad2) -> Net-(J75-Pad1)
- Q22 pad 1: Net-(D35-Pad2) -> Net-(J77-Pad1)
- Q23 pad 1: Net-(D37-Pad2) -> Net-(J81-Pad1)
- Q24 pad 1: Net-(D38-Pad2) -> Net-(J83-Pad1)
- Q3 pad 1: Net-(D7-Pad2) -> Net-(J21-Pad1)
- Q4 pad 1: Net-(D8-Pad2) -> Net-(J23-Pad1)
- Q5 pad 1: Net-(D10-Pad2) -> Net-(J27-Pad1)
- Q6 pad 1: Net-(D11-Pad2) -> Net-(J29-Pad1)
- Q7 pad 1: Net-(D13-Pad2) -> Net-(J33-Pad1)
- Q8 pad 1: Net-(D14-Pad2) -> Net-(J35-Pad1)
- Q9 pad 1: Net-(D16-Pad2) -> Net-(J39-Pad1)
- R11 pad 1: Net-(R11-Pad1) -> Net-(C9-Pad2)
- R12 pad 1: /Phases/A_VOLTAGE_SENSE -> Net-(J6-Pad1)
- R12 pad 2: /Phases/PHASE_A -> /GPIO0
- R13 pad 1: GNDA -> Net-(J6-Pad2)
- R13 pad 2: /Phases/A_VOLTAGE_SENSE -> /GPIO1
- R14 pad 1: /Phases/B_VOLTAGE_SENSE -> Net-(J6-Pad3)
- R14 pad 2: /Phases/PHASE_B -> /GPIO2
- R15 pad 1: GNDA -> Net-(J6-Pad4)
- R15 pad 2: /Phases/B_VOLTAGE_SENSE -> /GPIO3
- R16 pad 2: +3.3VA -> Net-(R16-Pad2)
- R17 pad 1: GNDA -> Net-(R17-Pad1)
- R18 pad 2: +3.3VA -> Net-(R18-Pad2)
- R19 pad 1: GNDA -> Net-(R19-Pad1)
- R20 pad 1: /Phases/C_VOLTAGE_SENSE -> Net-(R20-Pad1)
- R20 pad 2: /Phases/PHASE_C -> GND
- R21 pad 1: GNDA -> +3V3
- R21 pad 2: /Phases/C_VOLTAGE_SENSE -> Net-(R20-Pad1)
- R22 pad 2: Net-(R22-Pad2) -> Net-(C8-Pad2)
- R23 pad 2: Net-(R11-Pad1) -> Net-(C9-Pad2)
- R24 pad 1: /Supplies/VIN -> /QEI_A/HALL_A/GPIO0
- R24 pad 2: Net-(R24-Pad2) -> Net-(J7-Pad2)
- R25 pad 1: Net-(C16-Pad1) -> /QEI_B/HALL_B/GPIO1
- R25 pad 2: Net-(R25-Pad2) -> Net-(J7-Pad3)
- R26 pad 1: Net-(R25-Pad2) -> /HOME/HALL_C/GPIO2
- R26 pad 2: GND -> Net-(J7-Pad4)
- R27 pad 1: +5V -> +3V3
- R27 pad 2: Net-(L2-Pad1) -> Net-(J7-Pad2)
- R28 pad 1: Net-(R28-Pad1) -> +3V3
- R28 pad 2: GND -> Net-(J7-Pad3)
- R29 pad 1: Net-(R29-Pad1) -> +3V3
- R29 pad 2: Net-(L2-Pad1) -> Net-(J7-Pad4)
- R30 pad 1: +3V3 -> Net-(R16-Pad2)
- R30 pad 2: Net-(R28-Pad1) -> Net-(C12-Pad1)
- R31 pad 1: Net-(C22-Pad1) -> Net-(C12-Pad2)
- R31 pad 2: Net-(R31-Pad2) -> Net-(R17-Pad1)
- R32 pad 1: Net-(R31-Pad2) -> Net-(C13-Pad1)
- R32 pad 2: GND -> Net-(R18-Pad2)
- R57 pad 1: /Phases/A_CURRENT_SENSE -> Net-(J8-Pad1)
- R58 pad 1: /Phases/B_CURRENT_SENSE -> Net-(J9-Pad1)
- R9 pad 1: Net-(R22-Pad2) -> Net-(C8-Pad2)
- U1 pad 13: /Phases/C_VOLTAGE_SENSE -> /C_VOLTAGE_SENSE
- U1 pad 16: /HOME/HALL_C/GPIO2 -> /QEI_A/HALL_A/GPIO0
- U1 pad 17: unconnected-(U1-Pad17) -> /GPIO0
- U1 pad 18: unconnected-(U1-Pad18) -> /GPIO1
- U1 pad 19: unconnected-(U1-Pad19) -> /GPIO2
- U1 pad 20: unconnected-(U1-Pad20) -> /GPIO3
- U1 pad 29: /QEI_A/HALL_A/GPIO0 -> /QEI_B/HALL_B/GPIO1
- U1 pad 30: /QEI_B/HALL_B/GPIO1 -> /HOME/HALL_C/GPIO2
- U1 pad 8: /Phases/A_VOLTAGE_SENSE -> unconnected-(U1-Pad8)
- U1 pad 9: /Phases/B_VOLTAGE_SENSE -> unconnected-(U1-Pad9)
- U10 pad 6: /Phases/PHASE_A -> Net-(C30-Pad2)
- U11 pad 6: /Phases/PHASE_B -> Net-(C32-Pad2)
- U12 pad 6: /Phases/PHASE_B -> Net-(C34-Pad2)
- U13 pad 6: /Phases/PHASE_B -> Net-(C36-Pad2)
- U14 pad 6: /Phases/PHASE_B -> Net-(C38-Pad2)
- U15 pad 6: /Phases/PHASE_C -> Net-(C40-Pad2)
- U16 pad 6: /Phases/PHASE_C -> Net-(C42-Pad2)
- U17 pad 6: /Phases/PHASE_C -> Net-(C44-Pad2)
- U18 pad 6: /Phases/PHASE_C -> Net-(C46-Pad2)
- U2 pad 2: GNDA -> Net-(C12-Pad2)
- U2 pad 4: Net-(R22-Pad2) -> Net-(C8-Pad2)
- U2 pad 5: +3.3VA -> Net-(C12-Pad1)
- U3 pad 2: GNDA -> Net-(C13-Pad2)
- U3 pad 4: Net-(R11-Pad1) -> Net-(C9-Pad2)
- U3 pad 5: +3.3VA -> Net-(C13-Pad1)
- U4 pad 1: Net-(R24-Pad2) -> Net-(R20-Pad1)
- U4 pad 2: Net-(D1-Pad1) -> +3V3
- U4 pad 3: Net-(C15-Pad1) -> +5V
- U7 pad 6: /Phases/PHASE_A -> Net-(C24-Pad2)
- U8 pad 6: /Phases/PHASE_A -> Net-(C26-Pad2)
- U9 pad 6: /Phases/PHASE_A -> Net-(C28-Pad2)
Routing:
- net /Phases/PHASE_A: track 195.8 -> 0.00 mm, vias 63 -> 80
- net /Phases/PHASE_B: track 161.3 -> 0.00 mm, vias 61 -> 80
- net /Phases/PHASE_C: track 148.9 -> 0.00 mm, vias 62 -> 79
- net VDD: track 81.8 -> 0.00 mm, vias 46 -> 45
- net GNDA: track 80.1 -> 0.00 mm, vias 9 -> 0
- net GNDPWR: track 140.9 -> 68.4 mm, vias 58 -> 59
- net +3.3VA: track 70.5 -> 0.00 mm, vias 3 -> 2
- net Net-(D5-Pad2): track 54.8 -> 4.48 mm, vias 2 -> 0
- net Net-(D14-Pad2): track 53.7 -> 4.48 mm, vias 2 -> 0
- net Net-(D11-Pad2): track 53.4 -> 4.48 mm, vias 2 -> 0
- net Net-(D8-Pad2): track 53.3 -> 4.48 mm, vias 2 -> 0
- net /Phases/C_HIN: track 86.6 -> 38.5 mm, vias 6 -> 4
- net /Phases/~{C_LIN}: track 83.6 -> 35.5 mm, vias 6 -> 4
- net /Supplies/VIN: track 46.9 -> 0.00 mm
- net +3V3: track 86.5 -> 41.1 mm, vias 4 -> 0
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- added copper zone on F.Cu, net +12V
- added copper zone on In1.Cu, net VDD
- added copper zone on In2.Cu, net VDD
Other:
- board size 99.6 x 48.3 mm -> 86.4 x 48.3 mm
