File: esc/esc.kicad_pcb (KiCad board)
At the start: 4 copper layers, 86.4 x 48.3 mm, 252 parts, among them J10 Conn_01x01, J11 Conn_01x01, J12 Conn_01x01, J13 Conn_01x01, J14 Conn_01x01, J17 Conn_01x01, J18 Conn_01x01, J19 Conn_01x01, J20 Conn_01x01, J23 Conn_01x01, J24 Conn_01x01, J25 Conn_01x01, J26 Conn_01x01, J29 Conn_01x01, J3 Conn_01x05, J30 Conn_01x01, J31 Conn_01x01, J32 Conn_01x01, J35 Conn_01x01, J36 Conn_01x01, J37 Conn_01x01, J38 Conn_01x01, J41 Conn_01x01, J42 Conn_01x01, J43 Conn_01x01, J44 Conn_01x01, J47 Conn_01x01, J48 Conn_01x01, J49 Conn_01x01, J50 Conn_01x01, J53 Conn_01x01, J54 Conn_01x01, J55 Conn_01x01, J56 Conn_01x01, J59 Conn_01x01, J60 Conn_01x01, J61 Conn_01x01, J62 Conn_01x01, J65 Conn_01x01, J66 Conn_01x01, J67 Conn_01x01, J68 Conn_01x01, J7 Conn_01x05, J71 Conn_01x01, J72 Conn_01x01, J73 Conn_01x01, J74 Conn_01x01, J77 Conn_01x01, J78 Conn_01x01, J79 Conn_01x01, J8 Conn_01x01, J80 Conn_01x01, J83 Conn_01x01, J84 Conn_01x01, J85 Conn_01x01, J86 Conn_01x01, J87 Conn_01x01, J88 Conn_01x01, J89 Conn_01x01, J9 Conn_01x01, J90 Conn_01x01, J91 Conn_01x01, Q1 Q_NMOS_GDS, Q10 Q_NMOS_GDS, Q11 Q_NMOS_GDS, Q12 Q_NMOS_GDS, Q13 Q_NMOS_GDS, Q14 Q_NMOS_GDS, Q15 Q_NMOS_GDS, Q16 Q_NMOS_GDS, Q17 Q_NMOS_GDS, Q18 Q_NMOS_GDS, Q19 Q_NMOS_GDS, Q2 Q_NMOS_GDS, Q20 Q_NMOS_GDS, Q21 Q_NMOS_GDS, Q22 Q_NMOS_GDS, Q23 Q_NMOS_GDS, Q24 Q_NMOS_GDS, Q3 Q_NMOS_GDS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

Commit message: Pretty much finished new design
Parts:
- removed C10, C11, C14, C7: 1n, Capacitor_SMD:C_0603_1608Metric
- removed C18: 1u, Capacitor_SMD:C_0603_1608Metric
- removed C2, C5: 470u, footprints:HorizontalCap_10x16_P5
- removed J90, J91: Conn_01x01, Library:SmallPin
- removed NT1: NetTie_2, footprints:Nettie2
- removed R12, R13, R14, R15: 330, Resistor_SMD:R_0603_1608Metric
- removed TP1, TP2, TP4, TP5, TP6, TP7, TP8, TP9: TestPoint, TestPoint:TestPoint_Pad_1.0x1.0mm
- added J4: Conn_01x05, footprints:EdgeConnector_5, F.Cu at (117.5, 129.9)
- added J6: Conn_01x04, footprints:EdgeConnector_4, F.Cu at (128.1, 129.9)
- added R60: 0R, Resistor_SMD:R_0603_1608Metric, B.Cu at (113.8, 126.5)
- added R61: 0R, Resistor_SMD:R_0603_1608Metric, B.Cu at (113.8, 128.1)
- C1, C17, C22, C3, C4, C6, R1: moved to B.Cu
- J10, J11: footprint Library:SmallPin -> Library:SmallPad
- J3: footprint Connector_PinHeader_2.54mm:PinHeader_1x05_P2.54mm_Vertical -> footprints:ProgConnector
- J85, J87, J89: footprint Library:SmallPad -> Library:SmallPin
- moved C17 117.8 mm to (111.1, 127.1), turned to -90 degrees
- moved R24 108.3 mm to (119.8, 121.2), turned to 90 degrees
- moved C19 87.9 mm to (119.8, 124.3), turned to -90 degrees
- moved R25 87.2 mm to (121.4, 121.2), turned to 90 degrees
- moved R27 86.3 mm to (115.8, 85.5), turned to 180 degrees
- moved R26 85.0 mm to (123.1, 121.2), turned to 90 degrees
- moved C22 84.8 mm to (112.5, 85.6)
- moved C20 84.3 mm to (121.4, 124.3), turned to -90 degrees
- moved R29 76.7 mm to (121.9, 85.5)
- moved J3 75.2 mm to (136.9, 128.3), turned to 180 degrees
- moved C21 71.6 mm to (123.1, 124.3), turned to -90 degrees
- moved R28 68.0 mm to (118.9, 85.5), turned to 180 degrees
- moved J11 66.6 mm to (66.3, 124.5)
- moved R20 62.4 mm to (100.1, 126.7), turned to -90 degrees
- moved R21 60.2 mm to (100.1, 123.4), turned to -90 degrees
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Connections:
- net /HOME/HALL_C/GPIO2 renamed /HOME/HALL_C
- net /QEI_A/HALL_A/GPIO0 renamed /QEI_A/HALL_A
- net /QEI_B/HALL_B/GPIO1 renamed /QEI_B/HALL_B
- C12 pad 1: Net-(C12-Pad1) -> +3.3VA
- C12 pad 2: Net-(C12-Pad2) -> GNDA
- C13 pad 1: Net-(C13-Pad1) -> +3.3VA
- C13 pad 2: Net-(C13-Pad2) -> GNDA
- C23 pad 2: GNDPWR -> GND
- C25 pad 2: GNDPWR -> GND
- C27 pad 2: GNDPWR -> GND
- C29 pad 2: GNDPWR -> GND
- C31 pad 2: GNDPWR -> GND
- C33 pad 2: GNDPWR -> GND
- C35 pad 2: GNDPWR -> GND
- C37 pad 2: GNDPWR -> GND
- C39 pad 2: GNDPWR -> GND
- C41 pad 2: GNDPWR -> GND
- C43 pad 2: GNDPWR -> GND
- C45 pad 2: GNDPWR -> GND
- J10 pad 1: /Phases/A_CURRENT_SENSE -> /Phases/Phase B/BRIDGE_LOW
- J11 pad 1: /Phases/B_CURRENT_SENSE -> GNDPWR
- J8 pad 1: Net-(J8-Pad1) -> /Phases/Phase A/BRIDGE_LOW
- J84 pad 1: +3.3VA -> Net-(J84-Pad1)
- J85 pad 1: Net-(C13-Pad1) -> Net-(J85-Pad1)
- J86 pad 1: +3.3VA -> Net-(J86-Pad1)
- J87 pad 1: Net-(C12-Pad1) -> Net-(J87-Pad1)
- J88 pad 1: Net-(C12-Pad2) -> GNDPWR
- J89 pad 1: Net-(C13-Pad2) -> GND
- J9 pad 1: Net-(J9-Pad1) -> GNDPWR
- R10 pad 2: /Phases/Phase B/BRIDGE_LOW -> Net-(J86-Pad1)
- R11 pad 2: GNDPWR -> Net-(J87-Pad1)
- R30 pad 2: Net-(C12-Pad1) -> +3.3VA
- R31 pad 1: Net-(C12-Pad2) -> GNDA
- R32 pad 1: Net-(C13-Pad1) -> +3.3VA
- R57 pad 1: Net-(J8-Pad1) -> /Phases/A_CURRENT_SENSE
- R58 pad 1: Net-(J9-Pad1) -> /Phases/B_CURRENT_SENSE
- R59 pad 2: Net-(C13-Pad2) -> GNDA
- R8 pad 2: /Phases/Phase A/BRIDGE_LOW -> Net-(J84-Pad1)
- R9 pad 2: GNDPWR -> Net-(J85-Pad1)
- U1 pad 13: /C_VOLTAGE_SENSE -> unconnected-(U1-Pad13)
- U1 pad 21: /SPI_CLK -> /I2C_SCL
- U1 pad 24: /SPI_MISO -> /I2C_SDA
- U1 pad 25: /SPI_MOSI -> unconnected-(U1-Pad25)
- U1 pad 26: /SPI_SS -> unconnected-(U1-Pad26)
- U10 pad 4: GNDPWR -> GND
- U11 pad 4: GNDPWR -> GND
- U12 pad 4: GNDPWR -> GND
- U13 pad 4: GNDPWR -> GND
- U14 pad 4: GNDPWR -> GND
- U15 pad 4: GNDPWR -> GND
- U16 pad 4: GNDPWR -> GND
- U17 pad 4: GNDPWR -> GND
- U18 pad 4: GNDPWR -> GND
- U2 pad 2: Net-(C12-Pad2) -> GNDA
- U2 pad 5: Net-(C12-Pad1) -> +3.3VA
- U3 pad 2: Net-(C13-Pad2) -> GNDA
- U3 pad 5: Net-(C13-Pad1) -> +3.3VA
- U7 pad 4: GNDPWR -> GND
- U8 pad 4: GNDPWR -> GND
- U9 pad 4: GNDPWR -> GND
Routing:
- net +3V3: track 41.1 -> 127.7 mm, vias 0 -> 9
- net GND: track 32.7 -> 86.2 mm, vias 2 -> 25
- net +3.3VA: track 0.00 -> 51.0 mm, vias 2 -> 4
- net GNDPWR: track 68.4 -> 22.0 mm, vias 59 -> 51
- net GNDA: track 0.00 -> 34.6 mm, vias 0 -> 3
- net /Phases/~{A_LIN}: track 34.4 -> 67.9 mm, vias 4 -> 5
- net /Phases/A_HIN: track 36.2 -> 68.0 mm, vias 4 -> 5
- net /Phases/A_CURRENT_SENSE: track 0.00 -> 30.4 mm, vias 0 -> 2
- net +5V: track 0.00 -> 29.7 mm, vias 0 -> 1
- net /I2C_SCL: track 0.00 -> 23.6 mm, vias 0 -> 2
- net /I2C_SDA: track 0.00 -> 23.4 mm, vias 0 -> 2
- net /Phases/B_HIN: track 38.0 -> 57.5 mm, vias 4 -> 5
- net /QEI_B/HALL_B: track 0.00 -> 18.6 mm, vias 0 -> 1
- net +12V: track 70.8 -> 89.3 mm, vias 8 -> 13
- net /Phases/~{B_LIN}: track 35.3 -> 53.7 mm, vias 4 -> 5
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- added copper zone on In2.Cu, net /Phases/PHASE_A
- added copper zone on In2.Cu, net /Phases/PHASE_B
- added copper zone on In2.Cu, net /Phases/PHASE_C
- added copper zone on In1.Cu, net GNDA
- removed copper zone on F.Cu, net GND
- removed copper zone on In1.Cu, net GND
- removed copper zone on In2.Cu, net GNDA
- removed copper zone on In1.Cu, net GNDPWR
- removed copper zone on In2.Cu, net GNDPWR
Other:
- outline, holes or cut-outs redrawn

Commit message: (Tentatively) final design
Parts:
- added REF**: Mousebites_5mm, footprints:Mousebites_5mm, F.Cu at (95.8, 92.7)
- added REF**: Mousebites_5mm, footprints:Mousebites_5mm, F.Cu at (93.6, 92.7)
- added REF**: Mousebites_5mm, footprints:Mousebites_5mm, F.Cu at (95.8, 128.3)
- added REF**: Mousebites_5mm, footprints:Mousebites_5mm, F.Cu at (93.6, 128.3)
Routing:
- net VDD: vias 45 -> 69
Other:
- outline, holes or cut-outs redrawn
